Commit message: Fixed LIDAR issues

File: slam-ws/src/caffeine_description/urdf/caffeine.urdf.xacro (robot description, xacro)
@@ -262,5 +262,5 @@
    <link name="hokuyo_link">
       <visual>
-         <origin xyz="0 0 0" rpy="0 0 0"/>
+         <origin xyz="0 0 ${-hokuyo_height/2.0}" rpy="0 0 0"/>
          <geometry>
             <mesh filename="package://caffeine_description/urdf/meshes/hokuyo.dae"/>
@@ -268,5 +268,5 @@
       </visual>
       <collision>
-         <origin xyz="0 0 0" rpy="0 0 0"/>
+         <origin xyz="0 0 ${-hokuyo_height/2.0}" rpy="0 0 0"/>
          <geometry>
             <box size="${hokuyo_length} ${hokuyo_width} ${hokuyo_height}"/>
@@ -281,5 +281,5 @@
       <parent link="base_link"/>
       <child link="hokuyo_link"/>
-      <origin xyz="${-base_width/2.0} 0 ${base_height/2.0 + hokuyo_height/2.0}" rpy="0 0 0"/>
+      <origin xyz="${base_width/2.0} 0 ${base_height/2.0 + hokuyo_height/2.0 + hokuyo_height/2.0}" rpy="0 0 ${-135*pi/180}"/>
    </joint>
 </robot>
