Commit message: Currently using wrong dimensions & changed to effort controllers (this change fixed prev issue)

File: slam-ws/src/caffeine_description/urdf/caffeine.gazebo.xacro (robot description, xacro)
@@ -28,5 +28,5 @@
                         <robotBaseFrame>base_link</robotBaseFrame>
                         <torque>20</torque>
-                        <commandTopic>cmd_vel</commandTopic>
+                        <topicName>cmd_vel</topicName>
                         <odometryTopic>odom</odometryTopic>
                         <odometryFrame>odom</odometryFrame>
@@ -40,4 +40,5 @@
                 <plugin name="gazebo_ros_control" filename="libgazebo_ros_control.so">
                         <robotNamespace>caffeine</robotNamespace>
+                        <legacyModeNS>true</legacyModeNS>
                 </plugin>
         </gazebo>

File: slam-ws/src/caffeine_description/urdf/caffeine.urdf.xacro (robot description, xacro)
@@ -28,9 +28,9 @@
          <type>transmission_interface/SimpleTransmission</type>
          <joint name="${joint}">
-            <hardwareInterface>hardware_interface/PositionJointInterface</hardwareInterface>
+            <hardwareInterface>hardware_interface/EffortJointInterface</hardwareInterface>
             <mechanicalReduction>1</mechanicalReduction>
          </joint>
          <actuator name="${joint}_motor">
-            <hardwareInterface>hardware_interface/PositionJointInterface</hardwareInterface>
+            <hardwareInterface>hardware_interface/EffortJointInterface</hardwareInterface>
          </actuator>
       </transmission>

File: slam-ws/src/caffeine_description/urdf/constants.xacro (robot description, xacro)
@@ -2,11 +2,11 @@
 <robot name="constants" xmlns:xacro="http://ros.org/wiki/xacro">
    <!-- Constants for drivebase -->
-   <xacro:property name="base_length" value="0.3"/>
-   <xacro:property name="base_width" value="0.3"/>
-   <xacro:property name="base_height" value="0.15"/>
-   <xacro:property name="base_mass" value="3.0"/>
+   <xacro:property name="base_length" value="1.236"/>
+   <xacro:property name="base_width" value="0.703"/>
+   <xacro:property name="base_height" value="0.415"/>
+   <xacro:property name="base_mass" value="39.091"/>
    <!-- Constants for wheels -->
-   <xacro:property name="wheel_diam" value="0.1"/>
-   <xacro:property name="wheel_length" value="0.05"/>
+   <xacro:property name="wheel_diam" value="0.25"/>
+   <xacro:property name="wheel_length" value="0.09"/>
    <xacro:property name="wheel_mass" value="1.0"/>
    <xacro:property name="wheel_base_offset" value="0.02"/>

Commit message: SLAM-6: Added Hokuyo sensor to model

File: slam-ws/src/caffeine_description/urdf/caffeine.gazebo.xacro (robot description, xacro)
@@ -16,30 +16,64 @@
       <material>Gazebo/Black</material>
    </gazebo>
-        <gazebo>
-                <plugin name="caffeine_controller" filename="libgazebo_ros_skid_steer_drive.so">
-                        <updateRate>30.0</updateRate>
-                        <robotNamespace>caffeine</robotNamespace>
-                        <leftFrontJoint>left_front_wheel_joint</leftFrontJoint>
-                        <rightFrontJoint>right_front_wheel_joint</rightFrontJoint>
-                        <leftRearJoint>left_back_wheel_joint</leftRearJoint>
-                        <rightRearJoint>right_back_wheel_joint</rightRearJoint>
-                        <wheelSeparation>0.67</wheelSeparation>
-                        <wheelDiameter>0.1</wheelDiameter>
-                        <robotBaseFrame>base_link</robotBaseFrame>
-                        <torque>20</torque>
-                        <topicName>cmd_vel</topicName>
-                        <odometryTopic>odom</odometryTopic>
-                        <odometryFrame>odom</odometryFrame>
-                        <odometrySource>world</odometrySource>
-                        <publishOdomTF>true</publishOdomTF>
-                        <publishWheelJointState>true</publishWheelJointState>
-                        <broadcastTF>true</broadcastTF>
-                </plugin>
-        </gazebo>
-        <gazebo>
-                <plugin name="gazebo_ros_control" filename="libgazebo_ros_control.so">
-                        <robotNamespace>caffeine</robotNamespace>
-                        <legacyModeNS>true</legacyModeNS>
-                </plugin>
-        </gazebo>
+   <gazebo>
+      <plugin name="caffeine_controller" filename="libgazebo_ros_skid_steer_drive.so">
+         <updateRate>30.0</updateRate>
+         <robotNamespace>caffeine</robotNamespace>
+         <leftFrontJoint>left_front_wheel_joint</leftFrontJoint>
+         <rightFrontJoint>right_front_wheel_joint</rightFrontJoint>
+         <leftRearJoint>left_back_wheel_joint</leftRearJoint>
+         <rightRearJoint>right_back_wheel_joint</rightRearJoint>
+         <wheelSeparation>0.67</wheelSeparation>
+         <wheelDiameter>0.1</wheelDiameter>
+         <robotBaseFrame>base_link</robotBaseFrame>
+         <torque>20</torque>
+         <topicName>cmd_vel</topicName>
+         <odometryTopic>odom</odometryTopic>
+         <odometryFrame>odom</odometryFrame>
+         <odometrySource>world</odometrySource>
+         <publishOdomTF>true</publishOdomTF>
+         <publishWheelJointState>true</publishWheelJointState>
+         <broadcastTF>true</broadcastTF>
+      </plugin>
+   </gazebo>
+   <!-- IMPORTANT: Double check the numbers I'm using here with our actual sensor-->
+   <gazebo reference="hokuyo_link">
+      <sensor type="gpu_ray" name="hokuyo_sensor">
+         <pose>0 0 0 0 0 0</pose>
+         <visualize>false</visualize>
+         <update_rate>30</update_rate>
+         <ray>
+            <scan>
+               <horizontal>
+                  <samples>1080</samples>
+                  <resolution>1</resolution>
+                  <min_angle>0.0</min_angle>
+                  <max_angle>6.28</max_angle>
+               </horizontal>
+            </scan>
+            <range>
+               <min>0.01</min>
+               <max>5.6</max>
+               <resolution>0.01</resolution>
+            </range>
+            <noise>
+               <type>gaussian</type>
+               <!-- Noise based on gazebosim.org's tutorial on writing gazebo plugins w/ ROS. The comment they put will be reproduced:
+                    Noise parameters based on published spec for Hokuyo laser achieving "+-30mm" accuracy at range < 10 m. A mean of 0.0m and                     stddev of 0.01m will put 99.7% of samples within 0.03m of the true reading. -->
+               <mean>0.0</mean>
+               <stddev>0.01</stddev>
+            </noise>
+         </ray>
+         <plugin name="gazebo_ros_hokuyo_controller" filename="libgazebo_ros_gpu_laser.so">
+            <topicName>laserscan</topicName>
+            <frameName>hokuyo_link</frameName>
+         </plugin>
+      </sensor>
+   </gazebo>
+   <gazebo>
+      <plugin name="gazebo_ros_control" filename="libgazebo_ros_control.so">
+         <robotNamespace>caffeine</robotNamespace>
+         <legacyModeNS>true</legacyModeNS>
+      </plugin>
+   </gazebo>
 </robot>

File: slam-ws/src/caffeine_description/urdf/caffeine.urdf.xacro (robot description, xacro)
@@ -99,3 +99,27 @@
         </joint>
         <xacro:Transmission joint="left_back_wheel_joint"/>
+        <!-- Hokuyo sensor -->
+        <link name="hokuyo_link">
+           <collision>
+              <origin xyz="0 0 0" rpy="0 0 0"/>
+              <geometry>
+                 <box size="${hokuyo_length} ${hokuyo_width} ${hokuyo_height}"/>
+              </geometry>
+           </collision>
+           <visual>
+              <origin xyz="0 0 0" rpy="0 0 0"/>
+              <geometry>
+                 <mesh filename="package://caffeine_description/urdf/meshes/hokuyo.dae"/>
+              </geometry>
+           </visual>
+           <inertial>
+              <mass value="${hokuyo_mass}"/>
+              <xacro:box_inertia mass="${hokuyo_mass}" length="${hokuyo_length}" width="${hokuyo_width}" height="${hokuyo_height}"/>
+           </inertial>
+        </link>
+        <joint name="hokuyo_joint" type="fixed">
+           <parent link="base_link"/>
+           <child link="hokuyo_link"/>
+           <origin xyz="0 0 ${base_height/2.0}" rpy="0 0 0"/>
+        </joint>
 </robot>

File: slam-ws/src/caffeine_description/urdf/constants.xacro (robot description, xacro)
@@ -12,3 +12,8 @@
    <xacro:property name="wheel_base_offset" value="0.02"/>
    <xacro:property name="pi" value="3.1415926"/>
+   <!-- Constants for hokuyo sensor -->
+   <xacro:property name="hokuyo_length" value="0.05"/>
+   <xacro:property name="hokuyo_width" value="0.05"/>
+   <xacro:property name="hokuyo_height" value="0.07"/>
+   <xacro:property name="hokuyo_mass" value="0.16"/>
 </robot>

Commit message: Moving robot; casters moving unrealistically

File: slam-ws/src/caffeine_description/urdf/caffeine.gazebo.xacro (robot description, xacro)
@@ -31,5 +31,4 @@
       <material>Gazebo/Black</material>
    </gazebo>
-<!--
    <gazebo>
       <plugin name="caffeine_controller" filename="libgazebo_ros_diff_drive.so">
@@ -52,5 +51,4 @@
       </plugin>
    </gazebo>
--->
    <!-- IMPORTANT: Double check the numbers I'm using here with our actual sensor-->
    <gazebo reference="hokuyo_link">

File: slam-ws/src/caffeine_description/urdf/caffeine.urdf.xacro (robot description, xacro)
@@ -175,4 +175,14 @@
          </geometry>
       </visual>
+      <collision>
+         <origin rpy="0 0 0" xyz="0 0 0"/>
+         <geometry>
+            <box size="${gearbox_length} ${gearbox_width} ${gearbox_height}"/>
+         </geometry>
+      </collision>
+      <inertial>
+         <mass value="${gearbox_mass}"/>
+         <xacro:box_inertia mass="${gearbox_mass}" length="${gearbox_length}" width="${gearbox_width}" height="${gearbox_height}"/>
+      </inertial>
    </link>
    <joint name="right_motor_gearbox_housing_joint" type="fixed">
@@ -189,4 +199,14 @@
          </geometry>
       </visual>
+      <collision>
+         <origin rpy="0 0 0" xyz="0 0 0"/>
+         <geometry>
+            <box size="${gearbox_length} ${gearbox_width} ${gearbox_height}"/>
+         </geometry>
+      </collision>
+      <inertial>
+         <mass value="${gearbox_mass}"/>
+         <xacro:box_inertia mass="${gearbox_mass}" length="${gearbox_length}" width="${gearbox_width}" height="${gearbox_height}"/>
+      </inertial>
    </link>
    <joint name="left_motor_gearbox_housing_joint" type="fixed">
@@ -196,24 +216,23 @@
    </joint>
    <!-- Right wheel -->
- <!--  <link name="right_wheel">
+   <link name="right_wheel">
       <xacro:wheel_link_description />
    </link>
    <joint name="right_wheel_joint" type="continuous">
-      <axis xyz="0 0 1"/>
+      <axis xyz="0 1 0"/>
       <parent link="right_motor_gearbox_housing"/>
       <child link="right_wheel"/>
-      <origin rpy="0 0 0" xyz="0 ${gearbox_width/2.0} ${-gearbox_height}"/>
+      <origin rpy="0 0 0" xyz="0 ${gearbox_width/1.5} ${-gearbox_height}"/>
    </joint>
    <xacro:Transmission joint="right_wheel_joint"/>
--->
-   <!-- Right wheel -->
+   <!-- Left wheel -->
    <link name="left_wheel">
       <xacro:wheel_link_description />
    </link>
    <joint name="left_wheel_joint" type="continuous">
-      <axis xyz="0 0 1"/>
+      <axis xyz="0 1 0"/>
       <parent link="left_motor_gearbox_housing"/>
       <child link="left_wheel"/>
-      <origin rpy="0 0 0" xyz="0 ${-gearbox_width/2.0} ${-gearbox_height}"/>
+      <origin rpy="0 0 0" xyz="0 ${-gearbox_width/1.5} ${-gearbox_height}"/>
    </joint>
    <xacro:Transmission joint="left_wheel_joint"/>

File: slam-ws/src/caffeine_description/urdf/constants.xacro (robot description, xacro)
@@ -35,5 +35,6 @@
    <!-- Constants for the motor gearbox housing -->
    <xacro:property name="gearbox_height" value="0.102"/>
-   <xacro:property name="gearbox_width" value="0.101"/>
+   <xacro:property name="gearbox_width" value="0.191"/>
    <xacro:property name="gearbox_length" value="0.101"/>
+   <xacro:property name="gearbox_mass" value="0.1"/>
 </robot>

Commit message: Added LIDAR and Stand; LIDAR properties + location must be changed (self detection occuring)

File: slam-ws/src/caffeine_description/urdf/caffeine.gazebo.xacro (robot description, xacro)
@@ -31,4 +31,7 @@
       <material>Gazebo/Black</material>
    </gazebo>
+   <gazebo reference="stand">
+      <material>Gazebo/Green</material>
+   </gazebo>
    <gazebo>
       <plugin name="caffeine_controller" filename="libgazebo_ros_diff_drive.so">
@@ -53,7 +56,7 @@
    <!-- IMPORTANT: Double check the numbers I'm using here with our actual sensor-->
    <gazebo reference="hokuyo_link">
-      <sensor type="gpu_ray" name="hokuyo_sensor">
+      <sensor type="ray" name="hokuyo_sensor">
          <pose>0 0 0 0 0 0</pose>
-         <visualize>false</visualize>
+         <visualize>true</visualize>
          <update_rate>30</update_rate>
          <ray>
@@ -63,9 +66,9 @@
                   <resolution>1</resolution>
                   <min_angle>0.0</min_angle>
-                  <max_angle>6.28</max_angle>
+                  <max_angle>4.71</max_angle>
                </horizontal>
             </scan>
             <range>
-               <min>0.01</min>
+               <min>0.1</min>
                <max>5.6</max>
                <resolution>0.01</resolution>
@@ -79,6 +82,6 @@
             </noise>
          </ray>
-         <plugin name="gazebo_ros_hokuyo_controller" filename="libgazebo_ros_gpu_laser.so">
-            <topicName>laserscan</topicName>
+         <plugin name="gazebo_ros_hokuyo_controller" filename="libgazebo_ros_laser.so">
+            <topicName>scan</topicName>
             <frameName>hokuyo_link</frameName>
          </plugin>

File: slam-ws/src/caffeine_description/urdf/caffeine.urdf.xacro (robot description, xacro)
@@ -237,3 +237,49 @@
    </joint>
    <xacro:Transmission joint="left_wheel_joint"/>
+   <link name="stand">
+      <visual>
+         <origin rpy="0 0 0" xyz="0 0 ${stand_height/2.0}"/>
+         <geometry>
+            <box size="${stand_length} ${stand_width} ${stand_height}"/>
+         </geometry>
+      </visual>
+      <collision>
+         <origin rpy="0 0 0" xyz="0 0 ${stand_height/2.0}"/>
+         <geometry>
+            <box size="${stand_length} ${stand_width} ${stand_height}"/>
+         </geometry>
+      </collision>
+      <inertial>
+         <mass value="${stand_mass}"/>
+         <xacro:box_inertia mass="${stand_mass}" length="${stand_length}" width="${stand_width}" height="${stand_height}"/>
+      </inertial>
+   </link>
+   <joint name="stand_joint" type="fixed">
+      <parent link="base_link"/>
+      <child link="stand"/>
+      <origin rpy="0 0 0" xyz="0 0 0"/>
+   </joint>
+   <link name="hokuyo_link">
+      <visual>
+         <origin xyz="0 0 0" rpy="0 0 0"/>
+         <geometry>
+            <mesh filename="package://caffeine_description/urdf/meshes/hokuyo.dae"/>
+         </geometry>
+      </visual>
+      <collision>
+         <origin xyz="0 0 0" rpy="0 0 0"/>
+         <geometry>
+            <box size="${hokuyo_length} ${hokuyo_width} ${hokuyo_height}"/>
+         </geometry>
+      </collision>
+      <inertial>
+         <mass value="${hokuyo_mass}"/>
+         <xacro:box_inertia mass="${hokuyo_mass}" length="${hokuyo_length}" width="${hokuyo_width}" height="${hokuyo_height}"/>
+      </inertial>
+   </link>
+   <joint name="hokuyo_joint" type="fixed">
+      <parent link="base_link"/>
+      <child link="hokuyo_link"/>
+      <origin xyz="${-base_width/2.0} 0 ${base_height/2.0 + hokuyo_height/2.0}" rpy="0 0 0"/>
+   </joint>
 </robot>

File: slam-ws/src/caffeine_description/urdf/constants.xacro (robot description, xacro)
@@ -38,3 +38,8 @@
    <xacro:property name="gearbox_length" value="0.101"/>
    <xacro:property name="gearbox_mass" value="0.1"/>
+  <!-- Constants for the stands -->
+  <xacro:property name="stand_length" value="0.412"/>
+  <xacro:property name="stand_width" value="0.254"/>
+  <xacro:property name="stand_height" value="1.324"/>
+  <xacro:property name="stand_mass" value="1.0"/>
 </robot>
