Commit message: Currently not working commit. Done to transfer files to my other install

File: slam-ws/src/caffeine_description/urdf/caffeine.gazebo.xacro (robot description, xacro)
@@ -4,26 +4,41 @@
       <material>Gazebo/Purple</material>
    </gazebo>
-   <gazebo reference="right_front_wheel">
+   <gazebo reference="front_caster">
+      <material>Gazebo/Grey</material>
+   </gazebo>
+   <gazebo reference="back_caster">
+      <material>Gazebo/Grey</material>
+   </gazebo>
+   <gazebo reference="front_caster_wheel">
       <material>Gazebo/Black</material>
    </gazebo>
-   <gazebo reference="right_back_wheel">
+   <gazebo reference="back_caster_wheel">
       <material>Gazebo/Black</material>
    </gazebo>
-   <gazebo reference="left_front_wheel">
+   <gazebo reference="basement">
+      <material>Gazebo/Grey</material>
+   </gazebo>
+   <gazebo reference="right_motor_gearbox_housing">
+      <material>Gazebo/Grey</material>
+   </gazebo>
+   <gazebo reference="left_motor_gearbox_housing">
+      <material>Gazebo/Grey</material>
+   </gazebo>
+   <gazebo reference="left_wheel">
       <material>Gazebo/Black</material>
    </gazebo>
-   <gazebo reference="left_back_wheel">
+   <gazebo reference="right_wheel">
       <material>Gazebo/Black</material>
    </gazebo>
+<!--
    <gazebo>
-      <plugin name="caffeine_controller" filename="libgazebo_ros_skid_steer_drive.so">
+      <plugin name="caffeine_controller" filename="libgazebo_ros_diff_drive.so">
+         <alwaysOn>true</alwaysOn>
          <updateRate>30.0</updateRate>
          <robotNamespace>caffeine</robotNamespace>
-         <leftFrontJoint>left_front_wheel_joint</leftFrontJoint>
-         <rightFrontJoint>right_front_wheel_joint</rightFrontJoint>
-         <leftRearJoint>left_back_wheel_joint</leftRearJoint>
-         <rightRearJoint>right_back_wheel_joint</rightRearJoint>
-         <wheelSeparation>0.67</wheelSeparation>
-         <wheelDiameter>0.1</wheelDiameter>
+         <leftJoint>left_wheel_joint</leftJoint>
+         <rightJoint>right_wheel_joint</rightJoint>
+         <wheelSeparation>0.764</wheelSeparation>
+         <wheelDiameter>0.25</wheelDiameter>
          <robotBaseFrame>base_link</robotBaseFrame>
          <torque>20</torque>
@@ -37,4 +52,5 @@
       </plugin>
    </gazebo>
+-->
    <!-- IMPORTANT: Double check the numbers I'm using here with our actual sensor-->
    <gazebo reference="hokuyo_link">

File: slam-ws/src/caffeine_description/urdf/caffeine.urdf.xacro (robot description, xacro)
@@ -4,5 +4,24 @@
    <xacro:include filename="$(find caffeine_description)/urdf/caffeine.gazebo.xacro"/>
    <xacro:include filename="$(find caffeine_description)/urdf/constants.xacro"/>
-   <!-- xacro macro definitions for wheels -->
+   <!-- xacro macro definitions for caster wheels -->
+   <xacro:macro name="caster_wheel_link_description">
+      <visual>
+         <origin rpy="${pi/2} 0 0" xyz="0 0 0"/>
+         <geometry>
+            <cylinder length="${caster_wheel_length}" radius="${caster_wheel_diam/2.0}"/>
+         </geometry>
+      </visual>
+      <collision>
+         <origin rpy="${pi/2} 0 0" xyz="0 0 0"/>
+         <geometry>
+            <cylinder length="${caster_wheel_length}" radius="${caster_wheel_diam/2.0}"/>
+         </geometry>
+      </collision>
+      <inertial>
+        <mass value="${caster_wheel_mass}"/>
+        <xacro:cylinder_inertia mass="${caster_wheel_mass}" length="${caster_wheel_length}" radius="${caster_wheel_diam/2}"/>
+      </inertial>
+   </xacro:macro>
+   <!-- xacro macro for side wheels -->
    <xacro:macro name="wheel_link_description">
       <visual>
@@ -47,5 +66,5 @@
          <origin rpy="0 0 0" xyz="0 0 0"/>
          <geometry>
-            <box size="${base_length} ${base_width} ${base_height}"/>
+             <box size="${base_length} ${base_width} ${base_height}"/>
          </geometry>
       </collision>
@@ -55,71 +74,147 @@
       </inertial>
    </link>
-        <!-- Right front wheel -->
-        <link name="right_front_wheel">
-                <xacro:wheel_link_description />
-        </link>
-        <joint name="right_front_wheel_joint" type="continuous">
-                <parent link="base_link"/>
-                <child link="right_front_wheel"/>
-                <origin xyz="${base_length/3.0} ${-base_width/2.0 - wheel_base_offset} ${-base_height/2.5}" rpy="0 0 0"/>
-                <axis xyz="0 1 0"/>
-        </joint>
-        <xacro:Transmission joint="right_front_wheel_joint"/>
-        <!-- Right back wheel -->
-        <link name="right_back_wheel">
-                <xacro:wheel_link_description />
-        </link>
-        <joint name="right_back_wheel_joint" type="continuous">
-                <parent link="base_link"/>
-                <child link="right_back_wheel"/>
-                <origin xyz="${-base_length/3.0} ${-base_width/2.0 - wheel_base_offset} ${-base_height/2.5}" rpy="0 0 0"/>
-                <axis xyz="0 1 0"/>
-        </joint>
-        <xacro:Transmission joint="right_back_wheel_joint"/>
-        <!-- Left front wheel -->
-        <link name="left_front_wheel">
-                <xacro:wheel_link_description />
-        </link>
-        <joint name="left_front_wheel_joint" type="continuous">
-                <parent link="base_link"/>
-                <child link="left_front_wheel"/>
-                <origin xyz="${base_length/3.0} ${base_width/2.0 + wheel_base_offset} ${-base_height/2.5}" rpy="0 0 0"/>
-                <axis xyz="0 1 0"/>
-        </joint>
-        <xacro:Transmission joint="left_front_wheel_joint"/>
-        <!-- Left back wheel -->
-        <link name="left_back_wheel">
-                <xacro:wheel_link_description />
-        </link>
-        <joint name="left_back_wheel_joint" type="continuous">
-                <parent link="base_link"/>
-                <child link="left_back_wheel"/>
-                <origin xyz="${-base_length/3.0} ${base_width/2.0 + wheel_base_offset} ${-base_height/2.5}" rpy="0 0 0"/>
-                <axis xyz="0 1 0"/>
-        </joint>
-        <xacro:Transmission joint="left_back_wheel_joint"/>
-        <!-- Hokuyo sensor -->
-        <link name="hokuyo_link">
-           <collision>
-              <origin xyz="0 0 0" rpy="0 0 0"/>
-              <geometry>
-                 <box size="${hokuyo_length} ${hokuyo_width} ${hokuyo_height}"/>
-              </geometry>
-           </collision>
-           <visual>
-              <origin xyz="0 0 0" rpy="0 0 0"/>
-              <geometry>
-                 <mesh filename="package://caffeine_description/urdf/meshes/hokuyo.dae"/>
-              </geometry>
-           </visual>
-           <inertial>
-              <mass value="${hokuyo_mass}"/>
-              <xacro:box_inertia mass="${hokuyo_mass}" length="${hokuyo_length}" width="${hokuyo_width}" height="${hokuyo_height}"/>
-           </inertial>
-        </link>
-        <joint name="hokuyo_joint" type="fixed">
-           <parent link="base_link"/>
-           <child link="hokuyo_link"/>
-           <origin xyz="0 0 ${base_height/2.0}" rpy="0 0 0"/>
-        </joint>
+   <!-- Front caster -->
+   <link name="front_caster">
+      <visual>
+         <origin rpy="0 0 0" xyz="0 0 ${-caster_height/2.0}"/>
+         <geometry>
+            <box size="${caster_length} ${caster_width} ${caster_height}"/>
+         </geometry>
+      </visual>
+      <collision>
+         <origin rpy="0 0 0" xyz="0 0 ${-caster_height/2.0}"/>
+         <geometry>
+            <box size="${caster_length} ${caster_width} ${caster_height}"/>
+         </geometry>
+      </collision>
+      <inertial>
+         <mass value="${caster_mass}"/>
+         <xacro:box_inertia mass="${caster_mass}" length="${caster_length}" width="${caster_width}" height="${caster_height}"/>
+      </inertial>
+   </link>
+   <joint name="front_caster_joint" type="continuous">
+      <axis xyz="0 0 1"/>
+      <parent link="base_link"/>
+      <child link="front_caster"/>
+      <origin rpy="0 0 0" xyz="${caster_x} 0 ${caster_z}"/>
+   </joint>
+   <!-- Back caster -->
+   <link name="back_caster">
+      <visual>
+         <origin rpy="0 0 0" xyz="0 0 ${-caster_height/2.0}"/>
+         <geometry>
+            <box size="${caster_length} ${caster_width} ${caster_height}"/>
+         </geometry>
+      </visual>
+      <collision>
+         <origin rpy="0 0 0" xyz="0 0 ${-caster_height/2.0}"/>
+         <geometry>
+            <box size="${caster_length} ${caster_width} ${caster_height}"/>
+         </geometry>
+      </collision>
+      <inertial>
+         <mass value="${caster_mass}"/>
+         <xacro:box_inertia mass="${caster_mass}" length="${caster_length}" width="${caster_width}" height="${caster_height}"/>
+      </inertial>
+   </link>
+   <joint name="back_caster_joint" type="continuous">
+      <axis xyz="0 0 1"/>
+      <parent link="base_link"/>
+      <child link="back_caster"/>
+      <origin rpy="0 0 0" xyz="${-caster_x} 0 ${caster_z}"/>
+   </joint>
+   <!-- Front caster wheel -->
+   <link name="front_caster_wheel">
+      <xacro:caster_wheel_link_description />
+   </link>
+   <joint name="front_caster_wheel_joint" type="continuous">
+      <axis xyz="0 0 1"/>
+      <parent link="front_caster"/>
+      <child link="front_caster_wheel"/>
+      <origin rpy="0 0 0" xyz="0 0 ${caster_wheel_z}"/>
+   </joint>
+   <!-- Back caster wheel -->
+   <link name="back_caster_wheel">
+      <xacro:caster_wheel_link_description />
+   </link>
+   <joint name="back_caster_wheel_joint" type="continuous">
+      <axis xyz="0 0 1"/>
+      <parent link="back_caster"/>
+      <child link="back_caster_wheel"/>
+      <origin rpy="0 0 0" xyz="0 0 ${caster_wheel_z}"/>
+   </joint>
+   <!-- Basement -->
+   <link name="basement">
+      <visual>
+         <origin rpy="0 0 0" xyz="0 0 ${-basement_height/2.0}"/>
+         <geometry>
+            <box size="${basement_length} ${basement_width} ${basement_height}"/>
+         </geometry>
+      </visual>
+      <collision>
+         <origin rpy="0 0 0" xyz="0 0 0"/>
+         <geometry>
+            <box size="${basement_length} ${basement_width} ${basement_height}"/>
+         </geometry>
+      </collision>
+      <inertial>
+         <mass value="${basement_mass}"/>
+         <xacro:box_inertia mass="${basement_mass}" length="${basement_length}" width="${basement_width}" height="${basement_height}"/>
+      </inertial>
+   </link>
+   <joint name="basement_joint" type="fixed">
+      <parent link="base_link"/>
+      <child link="basement"/>
+   </joint>
+   <!-- Right side motor housing -->
+   <link name="right_motor_gearbox_housing">
+      <visual>
+         <origin rpy="0 0 0" xyz="0 0 ${-gearbox_height/2.0}"/>
+         <geometry>
+            <box size="${gearbox_length} ${gearbox_width} ${gearbox_height}"/>
+         </geometry>
+      </visual>
+   </link>
+   <joint name="right_motor_gearbox_housing_joint" type="fixed">
+      <parent link="base_link"/>
+      <child link="right_motor_gearbox_housing"/>
+      <origin rpy="0 0 0" xyz="0 ${base_length/4.0} 0"/>
+   </joint>
+   <!-- Left side motor housing -->
+   <link name="left_motor_gearbox_housing">
+      <visual>
+         <origin rpy="0 0 0" xyz="0 0 ${-gearbox_height/2.0}"/>
+         <geometry>
+            <box size="${gearbox_length} ${gearbox_width} ${gearbox_height}"/>
+         </geometry>
+      </visual>
+   </link>
+   <joint name="left_motor_gearbox_housing_joint" type="fixed">
+      <parent link="base_link"/>
+      <child link="left_motor_gearbox_housing"/>
+      <origin rpy="0 0 0" xyz="0 ${-base_length/4.0} 0"/>
+   </joint>
+   <!-- Right wheel -->
+ <!--  <link name="right_wheel">
+      <xacro:wheel_link_description />
+   </link>
+   <joint name="right_wheel_joint" type="continuous">
+      <axis xyz="0 0 1"/>
+      <parent link="right_motor_gearbox_housing"/>
+      <child link="right_wheel"/>
+      <origin rpy="0 0 0" xyz="0 ${gearbox_width/2.0} ${-gearbox_height}"/>
+   </joint>
+   <xacro:Transmission joint="right_wheel_joint"/>
+-->
+   <!-- Right wheel -->
+   <link name="left_wheel">
+      <xacro:wheel_link_description />
+   </link>
+   <joint name="left_wheel_joint" type="continuous">
+      <axis xyz="0 0 1"/>
+      <parent link="left_motor_gearbox_housing"/>
+      <child link="left_wheel"/>
+      <origin rpy="0 0 0" xyz="0 ${-gearbox_width/2.0} ${-gearbox_height}"/>
+   </joint>
+   <xacro:Transmission joint="left_wheel_joint"/>
 </robot>

File: slam-ws/src/caffeine_description/urdf/constants.xacro (robot description, xacro)
@@ -2,14 +2,25 @@
 <robot name="constants" xmlns:xacro="http://ros.org/wiki/xacro">
    <!-- Constants for drivebase -->
-   <xacro:property name="base_length" value="1.236"/>
-   <xacro:property name="base_width" value="0.703"/>
-   <xacro:property name="base_height" value="0.415"/>
+   <xacro:property name="base_length" value="1.268"/>
+   <xacro:property name="base_width" value="0.764"/>
+   <xacro:property name="base_height" value="0.01"/>
    <xacro:property name="base_mass" value="39.091"/>
-   <!-- Constants for wheels -->
+   <!-- Constants for caster wheels -->
+   <xacro:property name="caster_wheel_diam" value="0.15"/>
+   <xacro:property name="caster_wheel_length" value="0.045"/>
+   <xacro:property name="caster_wheel_mass" value="1.0"/>
+   <xacro:property name="pi" value="3.1415926"/>
+   <xacro:property name="caster_wheel_z" value="-0.141"/>
+   <!-- Constants for side wheels -->
    <xacro:property name="wheel_diam" value="0.25"/>
    <xacro:property name="wheel_length" value="0.09"/>
    <xacro:property name="wheel_mass" value="1.0"/>
-   <xacro:property name="wheel_base_offset" value="0.02"/>
-   <xacro:property name="pi" value="3.1415926"/>
+   <!-- Constants for casters -->
+   <xacro:property name="caster_length" value="0.113"/>
+   <xacro:property name="caster_width" value="0.089"/>
+   <xacro:property name="caster_height" value="0.141"/>
+   <xacro:property name="caster_x" value="0.578"/>
+   <xacro:property name="caster_z" value="-0.005"/>
+   <xacro:property name="caster_mass" value="1.0"/>
    <!-- Constants for hokuyo sensor -->
    <xacro:property name="hokuyo_length" value="0.05"/>
@@ -17,3 +28,12 @@
    <xacro:property name="hokuyo_height" value="0.07"/>
    <xacro:property name="hokuyo_mass" value="0.16"/>
+   <!-- Constants for the basement -->
+   <xacro:property name="basement_height" value="0.103"/>
+   <xacro:property name="basement_width" value="0.305"/>
+   <xacro:property name="basement_length" value="0.456"/>
+   <xacro:property name="basement_mass" value="1.0"/>
+   <!-- Constants for the motor gearbox housing -->
+   <xacro:property name="gearbox_height" value="0.102"/>
+   <xacro:property name="gearbox_width" value="0.101"/>
+   <xacro:property name="gearbox_length" value="0.101"/>
 </robot>

Commit message: Changedlaser frame name to base_laser

File: slam-ws/src/caffeine_description/urdf/caffeine.gazebo.xacro (robot description, xacro)
@@ -54,5 +54,5 @@
    </gazebo>
    <!-- IMPORTANT: Double check the numbers I'm using here with our actual sensor-->
-   <gazebo reference="hokuyo_link">
+   <gazebo reference="base_laser">
       <sensor type="ray" name="hokuyo_sensor">
          <pose>0 0 0 0 0 0</pose>
@@ -83,5 +83,5 @@
          <plugin name="gazebo_ros_hokuyo_controller" filename="libgazebo_ros_laser.so">
             <topicName>/scan</topicName>
-            <frameName>hokuyo_link</frameName>
+            <frameName>base_laser</frameName>
          </plugin>
       </sensor>

File: slam-ws/src/caffeine_description/urdf/caffeine.urdf.xacro (robot description, xacro)
@@ -260,5 +260,5 @@
       <origin rpy="0 0 0" xyz="0 0 0"/>
    </joint>
-   <link name="hokuyo_link">
+   <link name="base_laser">
       <visual>
          <origin xyz="0 0 ${-hokuyo_height/2.0}" rpy="0 0 0"/>
@@ -278,7 +278,7 @@
       </inertial>
    </link>
-   <joint name="hokuyo_joint" type="fixed">
-      <parent link="base_link"/>
-      <child link="hokuyo_link"/>
+   <joint name="base_laser_joint" type="fixed">
+      <parent link="base_link"/>
+      <child link="base_laser"/>
       <origin xyz="${base_width/2.0} 0 ${base_height/2.0 + hokuyo_height/2.0 + hokuyo_height/2.0}" rpy="0 0 ${-135*pi/180}"/>
    </joint>
