Commit message: Adding ZED constants

File: slam-ws/src/caffeine/urdf/constants.xacro (robot description, xacro)
@@ -48,3 +48,9 @@
   <xacro:property name="stand_height" value="1.324"/>
   <xacro:property name="stand_mass" value="1.0"/>
+  <!-- Constants for ZED camera -->
+  <!-- NOTE: approx as a rectangular prism -->
+  <xacro:property name="ZED_camera_mass" value="0.1587573"/>
+  <xacro:property name="ZED_camera_length" value="0.175"/>
+  <xacro:property name="ZED_camera_width" value="0.03"/>
+  <xacro:property name="ZED_camera_height" value="0.033"/>
 </robot>
