Commit message: Replacing tabs with 4 spaces

File: slam-ws/src/caffeine/urdf/inertias.xacro (robot description, xacro)
@@ -1,23 +1,23 @@
 <?xml version="1.0"?>
 <robot name="inertias" xmlns:xacro="http://ros.org/wiki/xacro">
-	<xacro:macro name="box_inertia" params="mass length width height">
-		<inertia
-			ixx="${mass * (height*height + length*length)/12.0}"
+    <xacro:macro name="box_inertia" params="mass length width height">
+        <inertia
+            ixx="${mass * (height*height + length*length)/12.0}"
                         ixy="0.0"
-			ixz="0.0"
+            ixz="0.0"
                         iyy="${mass * (width*width + length*length)/12.0}"
                         iyz="0.0"
-			izz="${mass * (width*width + height*height)/12.0}"
-		/>
-	</xacro:macro>
-	<xacro:macro name="cylinder_inertia" params="mass length radius">
-		<inertia
-			ixx="${mass * (3*radius*radius + length*length)/12.0}"
-			ixy="0.0"
-			ixz="0.0"
+            izz="${mass * (width*width + height*height)/12.0}"
+        />
+    </xacro:macro>
+    <xacro:macro name="cylinder_inertia" params="mass length radius">
+        <inertia
+            ixx="${mass * (3*radius*radius + length*length)/12.0}"
+            ixy="0.0"
+            ixz="0.0"
                         iyy="${mass * (3*radius*radius + length*length)/12.0}"
-			iyz="0.0"
-			izz="${0.5*mass*radius*radius}"
-		/>
-	</xacro:macro>
+            iyz="0.0"
+            izz="${0.5*mass*radius*radius}"
+        />
+    </xacro:macro>
 </robot>
