Commit message: Changed names from caffeine_description to caffeine

File: slam-ws/src/caffeine/urdf/caffeine.urdf.xacro (robot description, xacro)
@@ -1,7 +1,7 @@
 <?xml version="1.0"?>
 <robot name="caffeine" xmlns:xacro="http://ros.org/wiki/xacro">
-   <xacro:include filename="$(find caffeine_description)/urdf/inertias.xacro"/>
-   <xacro:include filename="$(find caffeine_description)/urdf/caffeine.gazebo.xacro"/>
-   <xacro:include filename="$(find caffeine_description)/urdf/constants.xacro"/>
+   <xacro:include filename="$(find caffeine)/urdf/inertias.xacro"/>
+   <xacro:include filename="$(find caffeine)/urdf/caffeine.gazebo.xacro"/>
+   <xacro:include filename="$(find caffeine)/urdf/constants.xacro"/>
    <!-- xacro macro definitions for caster wheels -->
    <xacro:macro name="caster_wheel_link_description">
@@ -264,5 +264,5 @@
          <origin xyz="0 0 ${-hokuyo_height/2.0}" rpy="0 0 0"/>
          <geometry>
-            <mesh filename="package://caffeine_description/urdf/meshes/hokuyo.dae"/>
+            <mesh filename="package://caffeine/urdf/meshes/hokuyo.dae"/>
          </geometry>
       </visual>

Commit message: HOTFIX: LIDAR veritcal offset

File: slam-ws/src/caffeine/urdf/caffeine.urdf.xacro (robot description, xacro)
@@ -283,5 +283,6 @@
       <parent link="base_link"/>
       <child link="base_laser"/>
-      <origin xyz="${base_width / 2.0} 0 ${base_height / 2.0 + hokuyo_height / 2.0}" rpy="0 0 ${-135 * pi / 180}"/>
+      <!-- HOTFIX: LIDAR offset-->
+      <origin xyz="${base_width / 2.0} 0 ${base_height / 2.0 + hokuyo_height / 2.0 + hokuyo_height / 2.0}" rpy="0 0 ${-135 * pi / 180}"/>
    </joint>
    <!-- IMU -->

Commit message: Fixed Shaking in scan and drifting of rover and covariance matrix issue

File: slam-ws/src/caffeine/urdf/caffeine.urdf.xacro (robot description, xacro)
@@ -283,5 +283,5 @@
       <parent link="base_link"/>
       <child link="base_laser"/>
-      <origin xyz="${base_width / 2.0} 0 ${base_height / 2.0 + hokuyo_height / 2.0}" rpy="0 0 ${-135 * pi / 180}"/>
+      <origin xyz="${base_width / 2.0} 0 ${base_height / 2.0 + hokuyo_height / 2.0 + 0.5}" rpy="0 0 ${-135 * pi / 180}"/>
    </joint>
    <!-- IMU -->

Commit message: Slam 65 - Caffeine + Husky working with Simulation (#71)
* Use IMU odometry with ekf node and not gazebo odom. Currently robot position is erratic

* Removing gravity

* Fixed Shaking in scan and drifting of rover and covariance matrix issue

* Husky works with Nav Stack and Gmapping (individually and together) while using odometry/filtered

Co-authored-by: Abijay1998 <abijay1998@gmail.com>

File: slam-ws/src/caffeine/urdf/caffeine.urdf.xacro (robot description, xacro)
@@ -283,6 +283,6 @@
       <parent link="base_link"/>
       <child link="base_laser"/>
-      <!-- HOTFIX: LIDAR offset-->
-      <origin xyz="${base_width / 2.0} 0 ${base_height / 2.0 + hokuyo_height / 2.0 + hokuyo_height / 2.0}" rpy="0 0 ${-135 * pi / 180}"/>
+      <!-- HOTFIX: LIDAR is not obstructed by the Caffeine itself -->
+      <origin xyz="${base_width / 2.0} 0 ${base_height / 2.0 + hokuyo_height / 2.0 + 0.5}" rpy="0 0 ${-135 * pi / 180}"/>
    </joint>
    <!-- IMU -->

Commit message: Adding sensor to urdf

File: slam-ws/src/caffeine/urdf/caffeine.urdf.xacro (robot description, xacro)
@@ -286,4 +286,45 @@
       <origin xyz="${base_width / 2.0} 0 ${base_height / 2.0 + hokuyo_height / 2.0 + 0.5}" rpy="0 0 ${-135 * pi / 180}"/>
    </joint>
+   <!-- ZED Camera -->
+  <link name="zed_camera_link">
+      <visual>
+         <origin xyz="0 0 0" rpy="0 0 0"/>
+            <!-- TODO: should be using the mesh but couldn't get it to work -->
+         <geometry>
+            <box size="${ZED_camera_length} ${ZED_camera_width} ${ZED_camera_height}"/>
+         </geometry>
+       </visual>
+       <collision>
+           <origin xyz="0 0 0" rpy="0 0 0"/>
+           <geometry>
+               <box size="${ZED_camera_length} ${ZED_camera_width} ${ZED_camera_height}"/>
+           </geometry>
+       </collision>
+       <inertial>
+           <mass value="${ZED_camera_mass}"/> <!-- Obtained from google search -->
+           <xacro:box_inertia mass="${ZED_camera_mass}" length="${ZED_camera_length}" width="${ZED_camera_width}" height="${ZED_camera_height}"/>
+       </inertial>
+   </link>
+   <joint name="zed_camera_joint" type="fixed">
+       <parent link="base_link"/>
+       <child link="zed_camera_link"/>
+       <origin xyz="${stand_length/2} 0 ${stand_height + ZED_camera_height}" rpy="${pi/4} 0 ${pi/2}"/>
+   </joint>
+   <!-- ZED camera lenses -->
+   <!-- NOTE: I'm only defining one and not visually showing any-->
+   <!-- I only need one for purposes of using the plugin -->
+   <!-- TODO: check if it's fine to call the left lense camera_link (rtabmap doesn't specify whether it wants the lense frame or the camera frame itself) -->
+   <link name="camera_link">
+       <!-- Inertial tag here to ensure that link does not phase through robot-->
+       <inertial>
+            <mass value="0.0001"/>
+            <inertia ixx="0.0001" ixy="0" ixz="0" iyy="0.0001" iyz="0" izz="0.00001"/>
+       </inertial>
+   </link>
+   <joint name="camera_link_joint" type="fixed">
+       <origin xyz="${ZED_camera_length/2.0} 0 0" rpy="0 0 ${3*pi/2}"/>
+       <parent link="zed_camera_link"/>
+       <child link="camera_link"/>
+   </joint>
    <!-- IMU -->
    <link name="imu_link">

Commit message: Added base_height/2 to zed camera joint height

File: slam-ws/src/caffeine/urdf/caffeine.urdf.xacro (robot description, xacro)
@@ -302,5 +302,5 @@
        </collision>
        <inertial>
-           <mass value="${ZED_camera_mass}"/> <!-- Obtained from google search -->
+           <mass value="${ZED_camera_mass}"/>
            <xacro:box_inertia mass="${ZED_camera_mass}" length="${ZED_camera_length}" width="${ZED_camera_width}" height="${ZED_camera_height}"/>
        </inertial>
@@ -309,5 +309,5 @@
        <parent link="base_link"/>
        <child link="zed_camera_link"/>
-       <origin xyz="${stand_length/2} 0 ${stand_height + ZED_camera_height}" rpy="${pi/4} 0 ${pi/2}"/>
+       <origin xyz="${stand_length/2} 0 ${stand_height + ZED_camera_height + base_height/2}" rpy="${pi/4} 0 ${pi/2}"/>
    </joint>
    <!-- ZED camera lenses -->

Commit message: Added filter to remove self-detection of lidar.

File: slam-ws/src/caffeine/urdf/caffeine.urdf.xacro (robot description, xacro)
@@ -284,5 +284,5 @@
       <child link="base_laser"/>
       <!-- HOTFIX: LIDAR is not obstructed by the Caffeine itself -->
-      <origin xyz="${base_width / 2.0} 0 ${base_height / 2.0 + hokuyo_height / 2.0 + 0.5}" rpy="0 0 ${-135 * pi / 180}"/>
+      <origin xyz="${base_width / 2.0} 0 ${base_height / 2.0 + hokuyo_height / 2.0}" rpy="0 0 0"/>
    </joint>
    <!-- ZED Camera -->

Commit message: Changed Visual Odom (zed) child_frame_id to use zed_camera_link. NOTE: need to add an offset to the Odom readings representative of the camera's location (only set for z value bc using 2d mode)

File: slam-ws/src/caffeine/urdf/caffeine.urdf.xacro (robot description, xacro)
@@ -287,5 +287,5 @@
    </joint>
    <!-- ZED Camera -->
-  <link name="zed_camera_link">
+   <link name="zed_camera_link">
       <visual>
          <origin xyz="0 0 0" rpy="0 0 0"/>

Commit message: Slam 72 - Added Laser FIltering Node to Prevent Self-Detection of the Robot. (#75)
* Added filter to remove self-detection of lidar.

* Cleanup.

* PR changes 1

Co-authored-by: Erick Mejia Uzeda <40526591+erickmu1@users.noreply.github.com>

File: slam-ws/src/caffeine/urdf/caffeine.urdf.xacro (robot description, xacro)
@@ -283,6 +283,5 @@
       <parent link="base_link"/>
       <child link="base_laser"/>
-      <!-- HOTFIX: LIDAR is not obstructed by the Caffeine itself -->
-      <origin xyz="${base_width / 2.0} 0 ${base_height / 2.0 + hokuyo_height / 2.0 + 0.5}" rpy="0 0 ${-135 * pi / 180}"/>
+      <origin xyz="${base_width / 2.0} 0 ${base_height / 2.0 + hokuyo_height / 2.0}" rpy="0 0 0"/>
    </joint>
    <!-- ZED Camera -->

Commit message: Moving camera to stand instead of base_link

File: slam-ws/src/caffeine/urdf/caffeine.urdf.xacro (robot description, xacro)
@@ -306,7 +306,7 @@
    </link>
    <joint name="zed_camera_joint" type="fixed">
-       <parent link="base_link"/>
+       <parent link="stand"/>
        <child link="zed_camera_link"/>
-       <origin xyz="${stand_length/2} 0 ${stand_height + ZED_camera_height + base_height/2}" rpy="0 ${pi/4} 0"/>
+       <origin xyz="${stand_length/2} 0 ${stand_height + ZED_camera_height}" rpy="0 0 0"/>
    </joint>
    <!-- ZED camera lenses -->

File: slam-ws/src/caffeine/urdf/constants.xacro (robot description, xacro)
@@ -10,5 +10,4 @@
    <xacro:property name="caster_wheel_length" value="0.045"/>
    <xacro:property name="caster_wheel_mass" value="1.0"/>
-   <xacro:property name="pi" value="3.1415926"/>
    <xacro:property name="caster_wheel_z" value="-0.141"/>
    <!-- Constants for side wheels -->
