Commit message: Added IMU link, joint, and Gazebo plugin. Need to use appropriate values

File: slam-ws/src/caffeine/urdf/caffeine.gazebo.xacro (robot description, xacro)
@@ -87,4 +87,24 @@
       </sensor>
    </gazebo>
+   <!-- TODO: Update values based on Phidget IMU specifications -->
+   <gazebo reference="imu_link">
+      <gravity>true</gravity>
+      <sensor name="imu_sensor" type="imu">
+         <always_on>true</always_on>
+         <update_rate>100</update_rate>
+         <visualize>true</visualize>
+         <topic>__default_topic__</topic>
+         <plugin filename="libgazebo_ros_imu_sensor.so" name="imu_plugin">
+            <topicName>imu</topicName>
+            <bodyName>imu_link</bodyName>
+            <updateRateHZ>10.0</updateRateHZ>
+            <gaussianNoise>0.0</gaussianNoise>
+            <xyzOffset>0 0 0</xyzOffset>
+            <rpyOffset>0 0 0</rpyOffset>
+            <frameName>imu_link</frameName>
+         </plugin>
+         <pose>0 0 0 0 0 0</pose>
+      </sensor>
+  </gazebo>
    <gazebo>
       <plugin name="gazebo_ros_control" filename="libgazebo_ros_control.so">

File: slam-ws/src/caffeine/urdf/caffeine.urdf.xacro (robot description, xacro)
@@ -260,4 +260,5 @@
       <origin rpy="0 0 0" xyz="0 0 0"/>
    </joint>
+   <!-- LIDAR -->
    <link name="base_laser">
       <visual>
@@ -283,3 +284,35 @@
       <origin xyz="${base_width/2.0} 0 ${base_height/2.0 + hokuyo_height/2.0 + hokuyo_height/2.0}" rpy="0 0 ${-135*pi/180}"/>
    </joint>
+   <!-- IMU -->
+   <link name="imu_link">
+      <inertial>
+         <origin xyz="0 0 0" rpy="0 0 0"/>
+         <mass value="0"/>
+         <inertia
+         ixx="1.0" ixy="0.0" ixz="0.0"
+         iyy="1.0" iyz="0.0"
+         izz="1.0"/>
+      </inertial>
+      <visual>
+         <origin xyz="0 0 0" rpy="0 0 0"/>
+         <geometry>
+            <box size="0.05 0.03 0.005"/>
+         </geometry>
+         <material name="green">
+            <color rgba="0 0.5 0 0.5"/>
+         </material>
+      </visual>
+      <collision>
+         <origin xyz="0 0 0" rpy="0 0 0"/>
+         <geometry>
+            <box size="0.05 0.03 0.005"/>
+         </geometry>
+      </collision>
+   </link>
+   <!-- Attach imu link to base link -->
+   <joint name="base_link_to_imu_link" type="fixed">
+      <parent link="base_link"/>
+      <child link="imu_link"/>
+      <origin xyz="0.1 -0.025 0.06" rpy="0 0 0"/>
+   </joint>
 </robot>

Commit message: Corrected IMU dimensions, transform, topic, and gave it appropriate colour

File: slam-ws/src/caffeine/urdf/caffeine.gazebo.xacro (robot description, xacro)
@@ -89,4 +89,5 @@
    <!-- TODO: Update values based on Phidget IMU specifications -->
    <gazebo reference="imu_link">
+      <material>Gazebo/Black</material>
       <gravity>true</gravity>
       <sensor name="imu_sensor" type="imu">
@@ -96,5 +97,5 @@
          <topic>__default_topic__</topic>
          <plugin filename="libgazebo_ros_imu_sensor.so" name="imu_plugin">
-            <topicName>imu</topicName>
+            <topicName>imu/data_raw</topicName>
             <bodyName>imu_link</bodyName>
             <updateRateHZ>10.0</updateRateHZ>

File: slam-ws/src/caffeine/urdf/caffeine.urdf.xacro (robot description, xacro)
@@ -262,57 +262,51 @@
    <!-- LIDAR -->
    <link name="base_laser">
-      <visual>
-         <origin xyz="0 0 ${-hokuyo_height/2.0}" rpy="0 0 0"/>
-         <geometry>
-            <mesh filename="package://caffeine/urdf/meshes/hokuyo.dae"/>
-         </geometry>
-      </visual>
-      <collision>
-         <origin xyz="0 0 ${-hokuyo_height/2.0}" rpy="0 0 0"/>
-         <geometry>
-            <box size="${hokuyo_length} ${hokuyo_width} ${hokuyo_height}"/>
-         </geometry>
-      </collision>
       <inertial>
          <mass value="${hokuyo_mass}"/>
          <xacro:box_inertia mass="${hokuyo_mass}" length="${hokuyo_length}" width="${hokuyo_width}" height="${hokuyo_height}"/>
       </inertial>
-   </link>
+      <visual>
+         <origin xyz="0 0 0" rpy="0 0 0"/>
+         <geometry>
+            <mesh filename="package://caffeine/urdf/meshes/hokuyo.dae"/>
+         </geometry>
+      </visual>
+      <collision>
+         <origin xyz="0 0 0" rpy="0 0 0"/>
+         <geometry>
+            <box size="${hokuyo_length} ${hokuyo_width} ${hokuyo_height}"/>
+         </geometry>
+      </collision>
+   </link>
+   <!-- LIDAR: attach base_laser to base_link -->
    <joint name="base_laser_joint" type="fixed">
       <parent link="base_link"/>
       <child link="base_laser"/>
-      <origin xyz="${base_width/2.0} 0 ${base_height/2.0 + hokuyo_height/2.0 + hokuyo_height/2.0}" rpy="0 0 ${-135*pi/180}"/>
+      <origin xyz="${base_width / 2.0} 0 ${base_height / 2.0 + hokuyo_height / 2.0}" rpy="0 0 ${-135 * pi / 180}"/>
    </joint>
    <!-- IMU -->
    <link name="imu_link">
       <inertial>
+         <mass value="${phidget_mass}"/>
+         <xacro:box_inertia mass="${phidget_mass}" length="${phidget_length}" width="${phidget_width}" height="${phidget_height}"/>
+      </inertial>
+      <visual>
          <origin xyz="0 0 0" rpy="0 0 0"/>
-         <mass value="0"/>
-         <inertia
-         ixx="1.0" ixy="0.0" ixz="0.0"
-         iyy="1.0" iyz="0.0"
-         izz="1.0"/>
-      </inertial>
-      <visual>
+         <geometry>
+            <box size="${phidget_length} ${phidget_width} ${phidget_height}"/>
+         </geometry>
+      </visual>
+      <collision>
          <origin xyz="0 0 0" rpy="0 0 0"/>
          <geometry>
-            <box size="0.05 0.03 0.005"/>
-         </geometry>
-         <material name="green">
-            <color rgba="0 0.5 0 0.5"/>
-         </material>
-      </visual>
-      <collision>
-         <origin xyz="0 0 0" rpy="0 0 0"/>
-         <geometry>
-            <box size="0.05 0.03 0.005"/>
-         </geometry>
-      </collision>
-   </link>
-   <!-- Attach imu link to base link -->
+            <box size="${phidget_length} ${phidget_width} ${phidget_height}"/>
+         </geometry>
+      </collision>
+   </link>
+   <!-- IMU: attach imu_link to base_link -->
    <joint name="base_link_to_imu_link" type="fixed">
       <parent link="base_link"/>
       <child link="imu_link"/>
-      <origin xyz="0.1 -0.025 0.06" rpy="0 0 0"/>
+      <origin xyz="${base_width / 2.0 - 0.1} 0 ${base_height / 2.0 + phidget_height / 2.0}" rpy="0 0 0"/>
    </joint>
 </robot>

File: slam-ws/src/caffeine/urdf/constants.xacro (robot description, xacro)
@@ -28,4 +28,9 @@
    <xacro:property name="hokuyo_height" value="0.07"/>
    <xacro:property name="hokuyo_mass" value="0.16"/>
+   <!-- Constants for Phidget IMU -->
+   <xacro:property name="phidget_length" value="0.04"/>
+   <xacro:property name="phidget_width" value="0.0375"/>
+   <xacro:property name="phidget_height" value="0.01"/>
+   <xacro:property name="phidget_mass" value="0.04"/>
    <!-- Constants for the basement -->
    <xacro:property name="basement_height" value="0.103"/>

Commit message: Slam 56 - Simulate IMU in Gazebo (#69)
* Added IMU link, joint, and Gazebo plugin. Need to use appropriate values

* Corrected IMU dimensions, transform, topic, and gave it appropriate colour

* Updated imu sensor gazebo plugin to moderately reflect Phidget sensor (accuracy could be improved)

* Updated caffeine_setup.launch to reflect existence of imu_link

File: slam-ws/src/caffeine/urdf/caffeine.gazebo.xacro (robot description, xacro)
@@ -87,4 +87,25 @@
       </sensor>
    </gazebo>
+   <!-- Phidgets IMU specifications -->
+   <gazebo reference="imu_link">
+      <material>Gazebo/Black</material>
+      <gravity>true</gravity>
+      <sensor name="imu_sensor" type="imu">
+         <always_on>true</always_on>
+         <update_rate>128</update_rate>
+         <visualize>true</visualize>
+         <topic>imu/data_raw</topic>
+         <plugin filename="libgazebo_ros_imu_sensor.so" name="imu_plugin">
+            <topicName>imu/data_raw</topicName>
+            <bodyName>imu_link</bodyName>
+            <updateRateHZ>128.0</updateRateHZ>
+            <gaussianNoise>0.59</gaussianNoise>
+            <xyzOffset>0 0 0</xyzOffset>
+            <rpyOffset>0 0 0</rpyOffset>
+            <frameName>imu_link</frameName>
+         </plugin>
+         <pose>0 0 0 0 0 0</pose>
+      </sensor>
+  </gazebo>
    <gazebo>
       <plugin name="gazebo_ros_control" filename="libgazebo_ros_control.so">

File: slam-ws/src/caffeine/urdf/caffeine.urdf.xacro (robot description, xacro)
@@ -260,26 +260,53 @@
       <origin rpy="0 0 0" xyz="0 0 0"/>
    </joint>
+   <!-- LIDAR -->
    <link name="base_laser">
-      <visual>
-         <origin xyz="0 0 ${-hokuyo_height/2.0}" rpy="0 0 0"/>
-         <geometry>
-            <mesh filename="package://caffeine/urdf/meshes/hokuyo.dae"/>
-         </geometry>
-      </visual>
-      <collision>
-         <origin xyz="0 0 ${-hokuyo_height/2.0}" rpy="0 0 0"/>
-         <geometry>
-            <box size="${hokuyo_length} ${hokuyo_width} ${hokuyo_height}"/>
-         </geometry>
-      </collision>
       <inertial>
          <mass value="${hokuyo_mass}"/>
          <xacro:box_inertia mass="${hokuyo_mass}" length="${hokuyo_length}" width="${hokuyo_width}" height="${hokuyo_height}"/>
       </inertial>
-   </link>
+      <visual>
+         <origin xyz="0 0 0" rpy="0 0 0"/>
+         <geometry>
+            <mesh filename="package://caffeine/urdf/meshes/hokuyo.dae"/>
+         </geometry>
+      </visual>
+      <collision>
+         <origin xyz="0 0 0" rpy="0 0 0"/>
+         <geometry>
+            <box size="${hokuyo_length} ${hokuyo_width} ${hokuyo_height}"/>
+         </geometry>
+      </collision>
+   </link>
+   <!-- LIDAR: attach base_laser to base_link -->
    <joint name="base_laser_joint" type="fixed">
       <parent link="base_link"/>
       <child link="base_laser"/>
-      <origin xyz="${base_width/2.0} 0 ${base_height/2.0 + hokuyo_height/2.0 + hokuyo_height/2.0}" rpy="0 0 ${-135*pi/180}"/>
+      <origin xyz="${base_width / 2.0} 0 ${base_height / 2.0 + hokuyo_height / 2.0}" rpy="0 0 ${-135 * pi / 180}"/>
+   </joint>
+   <!-- IMU -->
+   <link name="imu_link">
+      <inertial>
+         <mass value="${phidget_mass}"/>
+         <xacro:box_inertia mass="${phidget_mass}" length="${phidget_length}" width="${phidget_width}" height="${phidget_height}"/>
+      </inertial>
+      <visual>
+         <origin xyz="0 0 0" rpy="0 0 0"/>
+         <geometry>
+            <box size="${phidget_length} ${phidget_width} ${phidget_height}"/>
+         </geometry>
+      </visual>
+      <collision>
+         <origin xyz="0 0 0" rpy="0 0 0"/>
+         <geometry>
+            <box size="${phidget_length} ${phidget_width} ${phidget_height}"/>
+         </geometry>
+      </collision>
+   </link>
+   <!-- IMU: attach imu_link to base_link -->
+   <joint name="base_link_to_imu_link" type="fixed">
+      <parent link="base_link"/>
+      <child link="imu_link"/>
+      <origin xyz="${base_width / 2.0 - 0.1} 0 ${base_height / 2.0 + phidget_height / 2.0}" rpy="0 0 0"/>
    </joint>
 </robot>

Commit message: added gps simulation in caffeine

File: slam-ws/src/caffeine/urdf/caffeine.gazebo.xacro (robot description, xacro)
@@ -33,4 +33,7 @@
    <gazebo reference="stand">
       <material>Gazebo/Green</material>
+   </gazebo>
+   <gazebo reference="gps_link">
+      <material>blue</material>
    </gazebo>
    <gazebo>
@@ -92,3 +95,16 @@
       </plugin>
    </gazebo>
+   <gazebo>
+      <plugin name="gps_controller" filename="libhector_gazebo_ros_gps.so">
+         <alwayson>true</alwayson>
+         <updaterate>1.0</updaterate>
+         <bodyname>gps_link</bodyname>
+         <!-- <topicname>/fix</topicname>
+         <velocitytopicname>/fix_velocity</velocitytopicname> -->
+         <drift>5.0 5.0 5.0</drift>
+         <gaussiannoise>0.1 0.1 0.1</gaussiannoise>
+         <velocitydrift>0 0 0</velocitydrift>
+         <velocitygaussiannoise>0.1 0.1 0.1</velocitygaussiannoise>
+      </plugin>
+   </gazebo>
 </robot>

File: slam-ws/src/caffeine/urdf/caffeine.urdf.xacro (robot description, xacro)
@@ -237,4 +237,5 @@
    </joint>
    <xacro:Transmission joint="left_wheel_joint"/>
+   <!--stand-->
    <link name="stand">
       <visual>
@@ -260,4 +261,5 @@
       <origin rpy="0 0 0" xyz="0 0 0"/>
    </joint>
+   <!--base laser-->
    <link name="base_laser">
       <visual>
@@ -283,3 +285,27 @@
       <origin xyz="${base_width/2.0} 0 ${base_height/2.0 + hokuyo_height/2.0 + hokuyo_height/2.0}" rpy="0 0 ${-135*pi/180}"/>
    </joint>
+   <!--GPS-->
+   <link name="gps_link">
+      <visual>
+         <origin xyz="0 0 0" rpy="0 0 0"/>
+         <geometry>
+            <box size="${gps_length} ${gps_width} ${gps_height}"/>
+         </geometry>
+      </visual>
+      <collision>
+         <origin xyz="0 0 0" rpy="0 0 0"/>
+         <geometry>
+            <box size="${gps_length} ${gps_width} ${gps_height}"/>
+         </geometry>
+      </collision>
+      <inertial>
+         <mass value="${gps_mass}"/>
+         <xacro:box_inertia mass="${gps_mass}" length="${gps_length}" width="${gps_width}" height="${gps_height}"/>
+      </inertial>
+   </link>
+   <joint name="gps_joint" type="fixed">
+      <parent link="base_link"/>
+      <child link="gps_link"/>
+      <origin xyz="${-base_width/2.0} 0 ${base_height/2.0 + gps_height}" rpy="0 0 0"/>
+   </joint>
 </robot>

File: slam-ws/src/caffeine/urdf/constants.xacro (robot description, xacro)
@@ -43,3 +43,8 @@
   <xacro:property name="stand_height" value="1.324"/>
   <xacro:property name="stand_mass" value="1.0"/>
+  <!-- Constants for the GPS -->
+  <xacro:property name="gps_height" value="0.1"/>
+  <xacro:property name="gps_width" value="0.07"/>
+  <xacro:property name="gps_length" value="0.07"/>
+  <xacro:property name="gps_mass" value="0.5"/>
 </robot>

Commit message: Fixed orientation of point-cloud, now the focal distance needs to be adjusted I think

File: slam-ws/src/caffeine/urdf/caffeine.gazebo.xacro (robot description, xacro)
@@ -127,5 +127,5 @@
             <depthImageInfoTopicName>depth/camera_info</depthImageInfoTopicName>
             <pointCloudTopicName>depth/points</pointCloudTopicName>
-            <frameName>camera_link</frameName>
+            <frameName>camera_view_link</frameName>
             <hackBaseline>0.06</hackBaseline>
             <distortionK1>0.0</distortionK1>

File: slam-ws/src/caffeine/urdf/caffeine.urdf.xacro (robot description, xacro)
@@ -292,5 +292,5 @@
             <!-- TODO: should be using the mesh but couldn't get it to work -->
          <geometry>
-            <box size="${ZED_camera_length} ${ZED_camera_width} ${ZED_camera_height}"/>
+            <box size="${ZED_camera_width} ${ZED_camera_length} ${ZED_camera_height}"/>
          </geometry>
        </visual>
@@ -298,5 +298,5 @@
            <origin xyz="0 0 0" rpy="0 0 0"/>
            <geometry>
-               <box size="${ZED_camera_length} ${ZED_camera_width} ${ZED_camera_height}"/>
+               <box size="${ZED_camera_width} ${ZED_camera_length} ${ZED_camera_height}"/>
            </geometry>
        </collision>
@@ -309,5 +309,5 @@
        <parent link="base_link"/>
        <child link="zed_camera_link"/>
-       <origin xyz="${stand_length/2} 0 ${stand_height + ZED_camera_height + base_height/2}" rpy="${pi/4} 0 ${pi/2}"/>
+       <origin xyz="${stand_length/2} 0 ${stand_height + ZED_camera_height + base_height/2}" rpy="0 0 0"/>
    </joint>
    <!-- ZED camera lenses -->
@@ -323,8 +323,20 @@
    </link>
    <joint name="camera_link_joint" type="fixed">
-       <origin xyz="${ZED_camera_length/2.0} 0 0" rpy="0 0 ${3*pi/2}"/>
+       <origin xyz="${ZED_camera_length/2.0} 0 0" rpy="0 0 0"/>
        <parent link="zed_camera_link"/>
        <child link="camera_link"/>
    </joint>
+   <link name="camera_view_link">
+       <!-- Inertial tag here to ensure that link does not phase through robot-->
+       <inertial>
+            <mass value="0.0001"/>
+            <inertia ixx="0.0001" ixy="0" ixz="0" iyy="0.0001" iyz="0" izz="0.00001"/>
+       </inertial>
+   </link>
+   <joint name="camera_view_link_joint" type="fixed">
+       <origin xyz="0 0 0" rpy="${-pi/2} 0 ${-pi/2}"/>
+       <parent link="camera_link"/>
+       <child link="camera_view_link"/>
+   </joint>
    <!-- IMU -->
    <link name="imu_link">

Commit message: Fixed point cloud

File: slam-ws/src/caffeine/urdf/caffeine.gazebo.xacro (robot description, xacro)
@@ -128,5 +128,5 @@
             <pointCloudTopicName>depth/points</pointCloudTopicName>
             <frameName>camera_view_link</frameName>
-            <hackBaseline>0.06</hackBaseline>
+            <hackBaseline>${ZED_camera_length}</hackBaseline>
             <distortionK1>0.0</distortionK1>
             <distortionK2>0.0</distortionK2>

File: slam-ws/src/caffeine/urdf/caffeine.urdf.xacro (robot description, xacro)
@@ -309,5 +309,5 @@
        <parent link="base_link"/>
        <child link="zed_camera_link"/>
-       <origin xyz="${stand_length/2} 0 ${stand_height + ZED_camera_height + base_height/2}" rpy="0 0 0"/>
+       <origin xyz="${stand_length/2} 0 ${stand_height + ZED_camera_height + base_height/2}" rpy="0 ${pi/4} 0"/>
    </joint>
    <!-- ZED camera lenses -->

Commit message: Slightly modified code to reflect garmin more

File: slam-ws/src/caffeine/urdf/caffeine.gazebo.xacro (robot description, xacro)
@@ -95,16 +95,21 @@
       </plugin>
    </gazebo>
-   <gazebo>
+   <!-- For details about plugin, see: http://wiki.ros.org/hector_gazebo_plugins -->
+   <!-- TODO: update these parameters to match real life Garmin. See: http://static.garmin.com/pumac/425_TechnicalSpecification.pdf -->
+   <!-- For testing purposes, this is not accurate -->
+  <gazebo>
       <plugin name="gps_controller" filename="libhector_gazebo_ros_gps.so">
-         <alwayson>true</alwayson>
-         <updaterate>1.0</updaterate>
-         <bodyname>gps_link</bodyname>
-         <!-- <topicname>/fix</topicname>
-         <velocitytopicname>/fix_velocity</velocitytopicname> -->
-         <drift>5.0 5.0 5.0</drift>
-         <gaussiannoise>0.1 0.1 0.1</gaussiannoise>
-         <velocitydrift>0 0 0</velocitydrift>
-         <velocitygaussiannoise>0.1 0.1 0.1</velocitygaussiannoise>
+        <updateRate>40.0</updateRate>
+        <bodyName>gps_link</bodyName>
+        <frameId>gps_link</frameId>
+        <topicName>gps/fix</topicName>
+        <velocityTopicName>gps/fix_velocity</velocityTopicName>
+        <referenceHeading>0</referenceHeading>
+        <referenceAltitude>0</referenceAltitude>
+        <!-- TODO: change drift parameter & gaussian noise parameters -->
+	<!-- Also might need to add velocity drift & gaussian noise for  velocity -->
+        <drift>0.0001 0.0001 0.0001</drift>
+        <gaussianNoise>0.01 0.01 0.1</gaussianNoise>
       </plugin>
-   </gazebo>
+  </gazebo>
 </robot>

File: slam-ws/src/caffeine/urdf/caffeine.urdf.xacro (robot description, xacro)
@@ -285,27 +285,27 @@
       <origin xyz="${base_width/2.0} 0 ${base_height/2.0 + hokuyo_height/2.0 + hokuyo_height/2.0}" rpy="0 0 ${-135*pi/180}"/>
    </joint>
-   <!--GPS-->
-   <link name="gps_link">
-      <visual>
-         <origin xyz="0 0 0" rpy="0 0 0"/>
-         <geometry>
-            <box size="${gps_length} ${gps_width} ${gps_height}"/>
-         </geometry>
-      </visual>
-      <collision>
-         <origin xyz="0 0 0" rpy="0 0 0"/>
-         <geometry>
-            <box size="${gps_length} ${gps_width} ${gps_height}"/>
-         </geometry>
-      </collision>
-      <inertial>
-         <mass value="${gps_mass}"/>
-         <xacro:box_inertia mass="${gps_mass}" length="${gps_length}" width="${gps_width}" height="${gps_height}"/>
-      </inertial>
-   </link>
-   <joint name="gps_joint" type="fixed">
+  <!-- GPS -->
+  <link name="gps_link">
+      <inertial>
+          <mass value="${gps_mass}"/>
+          <xacro:cylinder_inertia mass="${gps_mass}" length="${gps_length}" radius="${gps_diam / 2.0}"/>
+      </inertial>
+      <visual>
+          <origin xyz="0 0 0" rpy="0 0 0"/>
+          <geometry>
+              <cylinder length="${gps_length}" radius="${gps_diam / 2.0}"/>
+          </geometry>
+      </visual>
+      <collision>
+          <origin xyz="0 0 0" rpy="0 0 0"/>
+          <geometry>
+              <cylinder length="${gps_length}" radius="${gps_diam / 2.0}"/>
+          </geometry>
+      </collision>
+  </link>
+  <joint name="gps_joint" type="fixed">
       <parent link="base_link"/>
       <child link="gps_link"/>
-      <origin xyz="${-base_width/2.0} 0 ${base_height/2.0 + gps_height}" rpy="0 0 0"/>
-   </joint>
+      <origin xyz="${-base_width / 2.0 - 0.1} 0 ${base_height / 2.0 + gps_length / 2.0}" rpy="0 0 0"/>
+  </joint>
 </robot>

File: slam-ws/src/caffeine/urdf/constants.xacro (robot description, xacro)
@@ -43,8 +43,8 @@
   <xacro:property name="stand_height" value="1.324"/>
   <xacro:property name="stand_mass" value="1.0"/>
-  <!-- Constants for the GPS -->
-  <xacro:property name="gps_height" value="0.1"/>
-  <xacro:property name="gps_width" value="0.07"/>
-  <xacro:property name="gps_length" value="0.07"/>
-  <xacro:property name="gps_mass" value="0.5"/>
+  <!-- Constants for Garmin GPS -->
+  <!-- NOTE: approx as a cylinder; garmin itself is similar to a hockey puck -->
+  <xacro:property name="gps_diam" value="0.061"/>
+  <xacro:property name="gps_length" value="0.0195"/>
+  <xacro:property name="gps_mass" value="0.165"/>
 </robot>
