Commit message: Added stereo camera orientation fix

File: slam-ws/src/caffeine/urdf/caffeine.gazebo.xacro (robot description, xacro)
@@ -127,5 +127,5 @@
             <pointCloudTopicName>depth/points</pointCloudTopicName>
             <frameName>camera_link</frameName>
-            <hackBaseline>0.06</hackBaseline>
+            <hackBaseline>${ZED_camera_length}</hackBaseline>
             <distortionK1>0.0</distortionK1>
             <distortionK2>0.0</distortionK2>

File: slam-ws/src/caffeine/urdf/caffeine.urdf.xacro (robot description, xacro)
@@ -291,5 +291,5 @@
             <!-- TODO: should be using the mesh but couldn't get it to work -->
          <geometry>
-            <box size="${ZED_camera_length} ${ZED_camera_width} ${ZED_camera_height}"/>
+            <box size="${ZED_camera_width} ${ZED_camera_length} ${ZED_camera_height}"/>
          </geometry>
        </visual>
@@ -297,5 +297,5 @@
            <origin xyz="0 0 0" rpy="0 0 0"/>
            <geometry>
-               <box size="${ZED_camera_length} ${ZED_camera_width} ${ZED_camera_height}"/>
+               <box size="${ZED_camera_width} ${ZED_camera_length} ${ZED_camera_height}"/>
            </geometry>
        </collision>
@@ -308,5 +308,5 @@
        <parent link="base_link"/>
        <child link="zed_camera_link"/>
-       <origin xyz="${stand_length/2} 0 ${stand_height + ZED_camera_height + base_height/2}" rpy="${pi/4} 0 ${pi/2}"/>
+       <origin xyz="${stand_length/2} 0 ${stand_height + ZED_camera_height + base_height/2}" rpy="0 ${pi/4} 0"/>
    </joint>
    <!-- ZED camera lenses -->
@@ -322,5 +322,5 @@
    </link>
    <joint name="camera_link_joint" type="fixed">
-       <origin xyz="${ZED_camera_length/2.0} 0 0" rpy="0 0 ${3*pi/2}"/>
+       <origin xyz="${ZED_camera_length/2.0} 0 0" rpy="0 0 0"/>
        <parent link="zed_camera_link"/>
        <child link="camera_link"/>

Commit message: Added gps to caffeine simulation

File: slam-ws/src/caffeine/urdf/caffeine.gazebo.xacro (robot description, xacro)
@@ -157,4 +157,23 @@
       </sensor>
   </gazebo>
+   <!-- For details about plugin, see: http://wiki.ros.org/hector_gazebo_plugins -->
+   <!-- TODO: update these parameters to match real life Garmin. See: http://static.garmin.com/pumac/425_TechnicalSpecification.pdf -->
+   <!-- For testing purposes, this is not accurate -->
+   <!-- Also, it was difficult to test this. It seems to work, but more testing MUST be done -->
+  <gazebo>
+      <plugin name="gps_controller" filename="libhector_gazebo_ros_gps.so">
+        <updateRate>40.0</updateRate>
+        <bodyName>gps_link</bodyName>
+        <frameId>gps_link</frameId>
+        <topicName>gps/fix</topicName>
+        <velocityTopicName>gps/fix_velocity</velocityTopicName>
+        <referenceHeading>0</referenceHeading>
+        <referenceAltitude>0</referenceAltitude>
+        <!-- TODO: change drift parameter & gaussian noise parameters -->
+	<!-- Also might need to add velocity drift & gaussian noise for  velocity -->
+        <drift>0.0001 0.0001 0.0001</drift>
+        <gaussianNoise>0.01 0.01 0.1</gaussianNoise>
+      </plugin>
+  </gazebo>
    <gazebo>
       <plugin name="gazebo_ros_control" filename="libgazebo_ros_control.so">

File: slam-ws/src/caffeine/urdf/caffeine.urdf.xacro (robot description, xacro)
@@ -351,3 +351,28 @@
       <origin xyz="${base_width / 2.0 - 0.1} 0 ${base_height / 2.0 + phidget_height / 2.0}" rpy="0 0 0"/>
    </joint>
+  <!-- GPS -->
+  <link name="gps_link">
+      <inertial>
+          <mass value="${gps_mass}"/>
+          <xacro:cylinder_inertia mass="${gps_mass}" length="${gps_length}" radius="${gps_diam / 2.0}"/>
+      </inertial>
+      <visual>
+          <origin xyz="0 0 0" rpy="0 0 0"/>
+          <geometry>
+              <cylinder length="${gps_length}" radius="${gps_diam / 2.0}"/>
+          </geometry>
+      </visual>
+      <collision>
+          <origin xyz="0 0 0" rpy="0 0 0"/>
+          <geometry>
+              <cylinder length="${gps_length}" radius="${gps_diam / 2.0}"/>
+          </geometry>
+      </collision>
+  </link>
+  <!-- GPS: attach gps_link to base_link -->
+  <joint name="gps_joint" type="fixed">
+      <parent link="base_link"/>
+      <child link="gps_link"/>
+      <origin xyz="${-base_width / 2.0 - 0.1} 0 ${base_height / 2.0 + gps_length / 2.0}" rpy="0 0 0"/>
+  </joint>
 </robot>

File: slam-ws/src/caffeine/urdf/constants.xacro (robot description, xacro)
@@ -54,3 +54,8 @@
   <xacro:property name="ZED_camera_width" value="0.03"/>
   <xacro:property name="ZED_camera_height" value="0.033"/>
+  <!-- Constants for Garmin GPS -->
+  <!-- NOTE: approx as a cylinder; garmin itself is similar to a hockey puck -->
+  <xacro:property name="gps_diam" value="0.061"/>
+  <xacro:property name="gps_length" value="0.0195"/>
+  <xacro:property name="gps_mass" value="0.165"/>
 </robot>

Commit message: Added new optical frame (zed_camera_link_optical)

File: slam-ws/src/caffeine/urdf/caffeine.gazebo.xacro (robot description, xacro)
@@ -128,5 +128,5 @@
             <depthImageInfoTopicName>depth/camera_info</depthImageInfoTopicName>
             <pointCloudTopicName>depth/points</pointCloudTopicName>
-            <frameName>camera_view_link</frameName>
+            <frameName>zed_camera_link_optical</frameName>
             <hackBaseline>${ZED_camera_length}</hackBaseline>
             <distortionK1>0.0</distortionK1>

File: slam-ws/src/caffeine/urdf/caffeine.urdf.xacro (robot description, xacro)
@@ -326,15 +326,12 @@
        <child link="camera_link"/>
    </joint>
-   <link name="camera_view_link">
-       <!-- Inertial tag here to ensure that link does not phase through robot-->
-       <inertial>
-            <mass value="0.0001"/>
-            <inertia ixx="0.0001" ixy="0" ixz="0" iyy="0.0001" iyz="0" izz="0.00001"/>
-       </inertial>
-   </link>
-   <joint name="camera_view_link_joint" type="fixed">
+   <!-- Generate an optical frame http://www.ros.org/reps/rep-0103.html#suffix-frames so that ros and opencv can operate on the camera frame correctly -->
+   <link name="zed_camera_link_optical">
+   </link>
+   <joint name="zed_camera_link_optical_joint" type="fixed">
+       <!-- Transform b/w standard and optical frame -->
        <origin xyz="0 0 0" rpy="${-pi/2} 0 ${-pi/2}"/>
-       <parent link="camera_link"/>
-       <child link="camera_view_link"/>
+       <parent link="zed_camera_link"/>
+       <child link="zed_camera_link_optical"/>
    </joint>
    <!-- IMU -->

Commit message: Currently model seems to work; file is written messy so must be cleaned as well

File: slam-ws/src/caffeine/urdf/caffeine.gazebo.xacro (robot description, xacro)
@@ -3,5 +3,5 @@
    <xacro:include filename="$(find caffeine)/urdf/constants.xacro"/>
    <gazebo reference="base_link">
-      <material>Gazebo/Purple</material>
+       <material>Gazebo/Purple</material>
    </gazebo>
    <gazebo reference="front_caster">

File: slam-ws/src/caffeine/urdf/caffeine.urdf.xacro (robot description, xacro)
@@ -1,390 +1,187 @@
 <?xml version="1.0"?>
 <robot name="caffeine" xmlns:xacro="http://ros.org/wiki/xacro">
-   <xacro:include filename="$(find caffeine)/urdf/inertias.xacro"/>
-   <xacro:include filename="$(find caffeine)/urdf/caffeine.gazebo.xacro"/>
-   <xacro:include filename="$(find caffeine)/urdf/constants.xacro"/>
-   <!-- xacro macro definitions for caster wheels -->
-   <xacro:macro name="caster_wheel_link_description">
-      <visual>
-         <origin rpy="${pi/2} 0 0" xyz="0 0 0"/>
-         <geometry>
-            <cylinder length="${caster_wheel_length}" radius="${caster_wheel_diam/2.0}"/>
-         </geometry>
-      </visual>
-      <collision>
-         <origin rpy="${pi/2} 0 0" xyz="0 0 0"/>
-         <geometry>
-            <cylinder length="${caster_wheel_length}" radius="${caster_wheel_diam/2.0}"/>
-         </geometry>
-      </collision>
-      <inertial>
-        <mass value="${caster_wheel_mass}"/>
-        <xacro:cylinder_inertia mass="${caster_wheel_mass}" length="${caster_wheel_length}" radius="${caster_wheel_diam/2}"/>
-      </inertial>
-   </xacro:macro>
-   <!-- xacro macro for side wheels -->
-   <xacro:macro name="wheel_link_description">
-      <visual>
-         <origin rpy="${pi/2} 0 0" xyz="0 0 0"/>
-         <geometry>
-            <cylinder length="${wheel_length}" radius="${wheel_diam/2.0}"/>
-         </geometry>
-      </visual>
-      <collision>
-         <origin rpy="${pi/2} 0 0" xyz="0 0 0"/>
-         <geometry>
-            <cylinder length="${wheel_length}" radius="${wheel_diam/2.0}"/>
-         </geometry>
-      </collision>
-      <inertial>
-        <mass value="${wheel_mass}"/>
-        <xacro:cylinder_inertia mass="${wheel_mass}" length="${wheel_length}" radius="${wheel_diam/2}"/>
-      </inertial>
-   </xacro:macro>
-   <!-- Wheel motor definitions -->
-   <xacro:macro name="Transmission" params="joint">
-      <transmission name="trans_${joint}">
-         <type>transmission_interface/SimpleTransmission</type>
-         <joint name="${joint}">
-            <hardwareInterface>hardware_interface/EffortJointInterface</hardwareInterface>
-            <mechanicalReduction>1</mechanicalReduction>
-         </joint>
-         <actuator name="${joint}_motor">
-            <hardwareInterface>hardware_interface/EffortJointInterface</hardwareInterface>
-         </actuator>
-      </transmission>
-   </xacro:macro>
-   <!-- Base link -->
-   <link name="base_link">
-      <visual>
-         <origin rpy="0 0 0" xyz="0 0 0"/>
-         <geometry>
-            <box size="${base_length} ${base_width} ${base_height}"/>
-         </geometry>
-      </visual>
-      <collision>
-         <origin rpy="0 0 0" xyz="0 0 0"/>
-         <geometry>
-             <box size="${base_length} ${base_width} ${base_height}"/>
-         </geometry>
-      </collision>
-      <inertial>
-         <mass value="${base_mass}"/>
-         <xacro:box_inertia mass="${base_mass}" length="${base_length}" width="${base_width}" height="${base_height}"/>
-      </inertial>
-   </link>
-   <!-- Front caster -->
-   <link name="front_caster">
-      <visual>
-         <origin rpy="0 0 0" xyz="0 0 ${-caster_height/2.0}"/>
-         <geometry>
-            <box size="${caster_length} ${caster_width} ${caster_height}"/>
-         </geometry>
-      </visual>
-      <collision>
-         <origin rpy="0 0 0" xyz="0 0 ${-caster_height/2.0}"/>
-         <geometry>
-            <box size="${caster_length} ${caster_width} ${caster_height}"/>
-         </geometry>
-      </collision>
-      <inertial>
-         <mass value="${caster_mass}"/>
-         <xacro:box_inertia mass="${caster_mass}" length="${caster_length}" width="${caster_width}" height="${caster_height}"/>
-      </inertial>
-   </link>
-   <joint name="front_caster_joint" type="continuous">
-      <axis xyz="0 0 1"/>
-      <parent link="base_link"/>
-      <child link="front_caster"/>
-      <origin rpy="0 0 0" xyz="${caster_x} 0 ${caster_z}"/>
-   </joint>
-   <!-- Back caster -->
-   <link name="back_caster">
-      <visual>
-         <origin rpy="0 0 0" xyz="0 0 ${-caster_height/2.0}"/>
-         <geometry>
-            <box size="${caster_length} ${caster_width} ${caster_height}"/>
-         </geometry>
-      </visual>
-      <collision>
-         <origin rpy="0 0 0" xyz="0 0 ${-caster_height/2.0}"/>
-         <geometry>
-            <box size="${caster_length} ${caster_width} ${caster_height}"/>
-         </geometry>
-      </collision>
-      <inertial>
-         <mass value="${caster_mass}"/>
-         <xacro:box_inertia mass="${caster_mass}" length="${caster_length}" width="${caster_width}" height="${caster_height}"/>
-      </inertial>
-   </link>
-   <joint name="back_caster_joint" type="continuous">
-      <axis xyz="0 0 1"/>
-      <parent link="base_link"/>
-      <child link="back_caster"/>
-      <origin rpy="0 0 0" xyz="${-caster_x} 0 ${caster_z}"/>
-   </joint>
-   <!-- Front caster wheel -->
-   <link name="front_caster_wheel">
-      <xacro:caster_wheel_link_description />
-   </link>
-   <joint name="front_caster_wheel_joint" type="continuous">
-      <axis xyz="0 0 1"/>
-      <parent link="front_caster"/>
-      <child link="front_caster_wheel"/>
-      <origin rpy="0 0 0" xyz="0 0 ${caster_wheel_z}"/>
-   </joint>
-   <!-- Back caster wheel -->
-   <link name="back_caster_wheel">
-      <xacro:caster_wheel_link_description />
-   </link>
-   <joint name="back_caster_wheel_joint" type="continuous">
-      <axis xyz="0 0 1"/>
-      <parent link="back_caster"/>
-      <child link="back_caster_wheel"/>
-      <origin rpy="0 0 0" xyz="0 0 ${caster_wheel_z}"/>
-   </joint>
-   <!-- Basement -->
-   <link name="basement">
-      <visual>
-         <origin rpy="0 0 0" xyz="0 0 ${-basement_height/2.0}"/>
-         <geometry>
-            <box size="${basement_length} ${basement_width} ${basement_height}"/>
-         </geometry>
-      </visual>
-      <collision>
-         <origin rpy="0 0 0" xyz="0 0 0"/>
-         <geometry>
-            <box size="${basement_length} ${basement_width} ${basement_height}"/>
-         </geometry>
-      </collision>
-      <inertial>
-         <mass value="${basement_mass}"/>
-         <xacro:box_inertia mass="${basement_mass}" length="${basement_length}" width="${basement_width}" height="${basement_height}"/>
-      </inertial>
-   </link>
-   <joint name="basement_joint" type="fixed">
-      <parent link="base_link"/>
-      <child link="basement"/>
-   </joint>
-   <!-- Right side motor housing -->
-   <link name="right_motor_gearbox_housing">
-      <visual>
-         <origin rpy="0 0 0" xyz="0 0 ${-gearbox_height/2.0}"/>
-         <geometry>
-            <box size="${gearbox_length} ${gearbox_width} ${gearbox_height}"/>
-         </geometry>
-      </visual>
-      <collision>
-         <origin rpy="0 0 0" xyz="0 0 0"/>
-         <geometry>
-            <box size="${gearbox_length} ${gearbox_width} ${gearbox_height}"/>
-         </geometry>
-      </collision>
-      <inertial>
-         <mass value="${gearbox_mass}"/>
-         <xacro:box_inertia mass="${gearbox_mass}" length="${gearbox_length}" width="${gearbox_width}" height="${gearbox_height}"/>
-      </inertial>
-   </link>
-   <joint name="right_motor_gearbox_housing_joint" type="fixed">
-      <parent link="base_link"/>
-      <child link="right_motor_gearbox_housing"/>
-      <origin rpy="0 0 0" xyz="0 ${base_length/4.0} 0"/>
-   </joint>
-   <!-- Left side motor housing -->
-   <link name="left_motor_gearbox_housing">
-      <visual>
-         <origin rpy="0 0 0" xyz="0 0 ${-gearbox_height/2.0}"/>
-         <geometry>
-            <box size="${gearbox_length} ${gearbox_width} ${gearbox_height}"/>
-         </geometry>
-      </visual>
-      <collision>
-         <origin rpy="0 0 0" xyz="0 0 0"/>
-         <geometry>
-            <box size="${gearbox_length} ${gearbox_width} ${gearbox_height}"/>
-         </geometry>
-      </collision>
-      <inertial>
-         <mass value="${gearbox_mass}"/>
-         <xacro:box_inertia mass="${gearbox_mass}" length="${gearbox_length}" width="${gearbox_width}" height="${gearbox_height}"/>
-      </inertial>
-   </link>
-   <joint name="left_motor_gearbox_housing_joint" type="fixed">
-      <parent link="base_link"/>
-      <child link="left_motor_gearbox_housing"/>
-      <origin rpy="0 0 0" xyz="0 ${-base_length/4.0} 0"/>
-   </joint>
-   <!-- Right wheel -->
-   <link name="right_wheel">
-      <xacro:wheel_link_description />
-   </link>
-   <joint name="right_wheel_joint" type="continuous">
-      <axis xyz="0 1 0"/>
-      <parent link="right_motor_gearbox_housing"/>
-      <child link="right_wheel"/>
-      <origin rpy="0 0 0" xyz="0 ${gearbox_width/1.5} ${-gearbox_height}"/>
-   </joint>
-   <xacro:Transmission joint="right_wheel_joint"/>
-   <!-- Left wheel -->
-   <link name="left_wheel">
-      <xacro:wheel_link_description />
-   </link>
-   <joint name="left_wheel_joint" type="continuous">
-      <axis xyz="0 1 0"/>
-      <parent link="left_motor_gearbox_housing"/>
-      <child link="left_wheel"/>
-      <origin rpy="0 0 0" xyz="0 ${-gearbox_width/1.5} ${-gearbox_height}"/>
-   </joint>
-   <xacro:Transmission joint="left_wheel_joint"/>
-   <link name="stand">
-      <visual>
-         <origin rpy="0 0 0" xyz="0 0 ${stand_height/2.0}"/>
-         <geometry>
-            <box size="${stand_length} ${stand_width} ${stand_height}"/>
-         </geometry>
-      </visual>
-      <collision>
-         <origin rpy="0 0 0" xyz="0 0 ${stand_height/2.0}"/>
-         <geometry>
-            <box size="${stand_length} ${stand_width} ${stand_height}"/>
-         </geometry>
-      </collision>
-      <inertial>
-         <mass value="${stand_mass}"/>
-         <xacro:box_inertia mass="${stand_mass}" length="${stand_length}" width="${stand_width}" height="${stand_height}"/>
-      </inertial>
-   </link>
-   <joint name="stand_joint" type="fixed">
-      <parent link="base_link"/>
-      <child link="stand"/>
-      <origin rpy="0 0 0" xyz="0 0 0"/>
-   </joint>
-   <!-- LIDAR -->
-   <link name="base_laser">
-      <inertial>
-         <mass value="${hokuyo_mass}"/>
-         <xacro:box_inertia mass="${hokuyo_mass}" length="${hokuyo_length}" width="${hokuyo_width}" height="${hokuyo_height}"/>
-      </inertial>
-      <visual>
-         <origin xyz="0 0 0" rpy="0 0 0"/>
-         <geometry>
-            <mesh filename="package://caffeine/urdf/meshes/hokuyo.dae"/>
-         </geometry>
-      </visual>
-      <collision>
-         <origin xyz="0 0 0" rpy="0 0 0"/>
-         <geometry>
-            <box size="${hokuyo_length} ${hokuyo_width} ${hokuyo_height}"/>
-         </geometry>
-      </collision>
-   </link>
-   <!-- LIDAR: attach base_laser to base_link -->
-   <joint name="base_laser_joint" type="fixed">
-      <parent link="base_link"/>
-      <child link="base_laser"/>
-      <origin xyz="${base_width / 2.0} 0 ${base_height / 2.0 + hokuyo_height / 2.0}" rpy="0 0 0"/>
-   </joint>
-   <!-- ZED Camera -->
-  <link name="zed_camera_link">
-      <visual>
-         <origin xyz="0 0 0" rpy="0 0 0"/>
-            <!-- TODO: should be using the mesh but couldn't get it to work -->
-         <geometry>
-            <box size="${ZED_camera_width} ${ZED_camera_length} ${ZED_camera_height}"/>
-         </geometry>
-       </visual>
-       <collision>
-           <origin xyz="0 0 0" rpy="0 0 0"/>
-           <geometry>
-               <box size="${ZED_camera_width} ${ZED_camera_length} ${ZED_camera_height}"/>
-           </geometry>
-       </collision>
-       <inertial>
-           <mass value="${ZED_camera_mass}"/>
-           <xacro:box_inertia mass="${ZED_camera_mass}" length="${ZED_camera_length}" width="${ZED_camera_width}" height="${ZED_camera_height}"/>
-       </inertial>
-   </link>
-   <joint name="zed_camera_joint" type="fixed">
-       <parent link="base_link"/>
-       <child link="zed_camera_link"/>
-       <origin xyz="${stand_length/2} 0 ${stand_height + ZED_camera_height + base_height/2}" rpy="0 ${pi/4} 0"/>
-   </joint>
-   <!-- ZED camera lenses -->
-   <!-- NOTE: I'm only defining one and not visually showing any-->
-   <!-- I only need one for purposes of using the plugin -->
-   <!-- TODO: check if it's fine to call the left lense camera_link (rtabmap doesn't specify whether it wants the lense frame or the camera frame itself) -->
-   <link name="camera_link">
-       <!-- Inertial tag here to ensure that link does not phase through robot-->
-       <inertial>
-            <mass value="0.0001"/>
-            <inertia ixx="0.0001" ixy="0" ixz="0" iyy="0.0001" iyz="0" izz="0.00001"/>
-       </inertial>
-   </link>
-   <joint name="camera_link_joint" type="fixed">
-       <origin xyz="${ZED_camera_length/2.0} 0 0" rpy="0 0 0"/>
-       <parent link="zed_camera_link"/>
-       <child link="camera_link"/>
-   </joint>
-   <link name="camera_view_link">
-       <!-- Inertial tag here to ensure that link does not phase through robot-->
-       <inertial>
-            <mass value="0.0001"/>
-            <inertia ixx="0.0001" ixy="0" ixz="0" iyy="0.0001" iyz="0" izz="0.00001"/>
-       </inertial>
-   </link>
-   <joint name="camera_view_link_joint" type="fixed">
-       <origin xyz="0 0 0" rpy="${-pi/2} 0 ${-pi/2}"/>
-       <parent link="camera_link"/>
-       <child link="camera_view_link"/>
-   </joint>
-   <!-- IMU -->
-   <link name="imu_link">
-      <inertial>
-         <mass value="${phidget_mass}"/>
-         <xacro:box_inertia mass="${phidget_mass}" length="${phidget_length}" width="${phidget_width}" height="${phidget_height}"/>
-      </inertial>
-      <visual>
-         <origin xyz="0 0 0" rpy="0 0 0"/>
-         <geometry>
-            <box size="${phidget_length} ${phidget_width} ${phidget_height}"/>
-         </geometry>
-      </visual>
-      <collision>
-         <origin xyz="0 0 0" rpy="0 0 0"/>
-         <geometry>
-            <box size="${phidget_length} ${phidget_width} ${phidget_height}"/>
-         </geometry>
-      </collision>
-   </link>
-   <!-- IMU: attach imu_link to base_link -->
-   <joint name="base_link_to_imu_link" type="fixed">
-      <parent link="base_link"/>
-      <child link="imu_link"/>
-      <origin xyz="${base_width / 2.0 - 0.1} 0 ${base_height / 2.0 + phidget_height / 2.0}" rpy="0 0 0"/>
-   </joint>
-  <!-- GPS -->
-  <link name="gps_link">
-      <inertial>
-          <mass value="${gps_mass}"/>
-          <xacro:cylinder_inertia mass="${gps_mass}" length="${gps_length}" radius="${gps_diam / 2.0}"/>
-      </inertial>
-      <visual>
-          <origin xyz="0 0 0" rpy="0 0 0"/>
-          <geometry>
-              <cylinder length="${gps_length}" radius="${gps_diam / 2.0}"/>
-          </geometry>
-      </visual>
-      <collision>
-          <origin xyz="0 0 0" rpy="0 0 0"/>
-          <geometry>
-              <cylinder length="${gps_length}" radius="${gps_diam / 2.0}"/>
-          </geometry>
-      </collision>
-  </link>
-  <!-- GPS: attach gps_link to base_link -->
-  <joint name="gps_joint" type="fixed">
-      <parent link="base_link"/>
-      <child link="gps_link"/>
-      <origin xyz="${-base_width / 2.0 - 0.1} 0 ${base_height / 2.0 + gps_length / 2.0}" rpy="0 0 0"/>
-  </joint>
+    <xacro:include filename="$(find caffeine)/urdf/inertias.xacro"/>
+    <xacro:include filename="$(find caffeine)/urdf/constants.xacro"/>
+    <xacro:include filename="$(find caffeine)/urdf/caffeine.gazebo.xacro"/>
+    <xacro:macro name="Transmission" params="joint">
+        <transmission name="trans_${joint}">
+            <type>transmission_interface/SimpleTransmission</type>
+            <joint name="${joint}">
+                <hardwareInterface>hardware_interface/EffortJointInterface</hardwareInterface>
+                <mechanicalReduction>1</mechanicalReduction>
+            </joint>
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