Commit message: Working caffeine model; IMU currently untested

File: slam-ws/src/caffeine/urdf/caffeine.gazebo.xacro (robot description, xacro)
@@ -2,37 +2,4 @@
 <robot name="caffeine_sim" xmlns:xacro="http://ros.org/wiki/xacro">
    <xacro:include filename="$(find caffeine)/urdf/constants.xacro"/>
-   <gazebo reference="base_link">
-       <material>Gazebo/Purple</material>
-   </gazebo>
-   <gazebo reference="front_caster">
-      <material>Gazebo/Grey</material>
-   </gazebo>
-   <gazebo reference="back_caster">
-      <material>Gazebo/Grey</material>
-   </gazebo>
-   <gazebo reference="front_caster_wheel">
-      <material>Gazebo/Black</material>
-   </gazebo>
-   <gazebo reference="back_caster_wheel">
-      <material>Gazebo/Black</material>
-   </gazebo>
-   <gazebo reference="basement">
-      <material>Gazebo/Grey</material>
-   </gazebo>
-   <gazebo reference="right_motor_gearbox_housing">
-      <material>Gazebo/Grey</material>
-   </gazebo>
-   <gazebo reference="left_motor_gearbox_housing">
-      <material>Gazebo/Grey</material>
-   </gazebo>
-   <gazebo reference="left_wheel">
-      <material>Gazebo/Black</material>
-   </gazebo>
-   <gazebo reference="right_wheel">
-      <material>Gazebo/Black</material>
-   </gazebo>
-   <gazebo reference="stand">
-      <material>Gazebo/Green</material>
-   </gazebo>
    <gazebo>
       <plugin name="caffeine_controller" filename="libgazebo_ros_diff_drive.so">
@@ -42,6 +9,6 @@
          <leftJoint>left_wheel_joint</leftJoint>
          <rightJoint>right_wheel_joint</rightJoint>
-         <wheelSeparation>0.764</wheelSeparation>
-         <wheelDiameter>0.25</wheelDiameter>
+         <wheelSeparation>${wheel_separation}</wheelSeparation>
+         <wheelDiameter>${wheel_diam}</wheelDiameter>
          <robotBaseFrame>base_link</robotBaseFrame>
          <torque>20</torque>
@@ -59,5 +26,5 @@
       <sensor type="ray" name="hokuyo_sensor">
          <pose>0 0 0 0 0 0</pose>
-         <visualize>false</visualize>
+         <visualize>true</visualize>
          <update_rate>30</update_rate>
          <ray>
@@ -66,6 +33,6 @@
                   <samples>1080</samples>
                   <resolution>1</resolution>
-                  <min_angle>0.0</min_angle>
-                  <max_angle>4.71</max_angle>
+                  <min_angle>-2.356</min_angle>
+                  <max_angle>2.356</max_angle>
                </horizontal>
             </scan>

File: slam-ws/src/caffeine/urdf/caffeine.urdf.xacro (robot description, xacro)
@@ -1,7 +1,7 @@
 <?xml version="1.0"?>
 <robot name="caffeine" xmlns:xacro="http://ros.org/wiki/xacro">
-    <xacro:include filename="$(find caffeine)/urdf/inertias.xacro"/>
     <xacro:include filename="$(find caffeine)/urdf/constants.xacro"/>
     <xacro:include filename="$(find caffeine)/urdf/caffeine.gazebo.xacro"/>
+    <xacro:include filename="$(find caffeine)/urdf/inertias.xacro"/>
     <xacro:macro name="Transmission" params="joint">
         <transmission name="trans_${joint}">
@@ -18,21 +18,37 @@
     <!-- Base link -->
     <link name="base_link">
-        <visual>
-            <origin rpy="0 0 0" xyz="0 0 0"/>
-            <geometry>
-                <mesh filename="package://caffeine/urdf/meshes/base_link.dae"/>
-            </geometry>
-        </visual>
-        <collision>
-            <origin rpy="0 0 0" xyz="0 0 0"/>
-            <geometry>
-                <mesh filename="package://caffeine/urdf/meshes/base_link.dae"/>
-            </geometry>
-        </collision>
-        <inertial>
-            <mass value="30"/>
-            <xacro:box_inertia mass="30" length="1" width="1" height="1"/>
-        </inertial>
-    </link>
+    </link>
+    <!-- Chassis link -->
+    <link name="chassis_link">
+        <visual>
+            <origin rpy="0 0 0" xyz="0 0 0"/>
+            <geometry>
+                <mesh filename="package://caffeine/urdf/meshes/chassis_link.dae"/>
+            </geometry>
+        </visual>
+        <collision>
+            <origin rpy="0 0 0" xyz="0 0 0"/>
+            <geometry>
+                <mesh filename="package://caffeine/urdf/meshes/chassis_link.dae"/>
+            </geometry>
+        </collision>
+        <inertial>
+            <mass value="${chassis_link_mass}"/>
+            <xacro:chassis_link_inertia/>
+        </inertial>
+    </link>
+    <joint name="chassis_link_joint" type="fixed">
+        <parent link="base_link"/>
+        <child link="chassis_link"/>
+        <origin rpy="0 0 0" xyz="0 0 ${base_link_z}"/>
+    </joint>
+    <!-- Stand link -->
+    <link name="stand_link">
+    </link>
+    <joint name="stand_link_joint" type="fixed">
+        <parent link="chassis_link"/>
+        <child link="stand_link"/>
+        <origin rpy="0 0 0" xyz="0 0 ${stand_link_z}"/>
+    </joint>
     <!-- Left wheel -->
     <link name="left_wheel">
@@ -51,15 +67,15 @@
         <inertial>
             <mass value="${wheel_mass}"/>
-            <xacro:cylinder_inertia mass="${wheel_mass}" length="${wheel_length}" radius="${wheel_diam/2.0}"/>
+            <xacro:wheel_inertia/>
         </inertial>
     </link>
     <joint name="left_wheel_joint" type="continuous">
         <axis xyz="0 1 0"/>
-        <parent link="base_link"/>
+        <parent link="chassis_link"/>
         <child link="left_wheel"/>
-        <origin rpy="0 0 0" xyz="0 0.43751887 -0.61759696"/>
+        <origin rpy="0 0 0" xyz="0 ${left_wheel_y} ${wheel_z}"/>
     </joint>
     <xacro:Transmission joint="left_wheel_joint"/>
-    <!-- RIght wheel -->
+    <!-- Right wheel -->
     <link name="right_wheel">
         <visual>
@@ -77,12 +93,12 @@
         <inertial>
             <mass value="${wheel_mass}"/>
-            <xacro:cylinder_inertia mass="${wheel_mass}" length="${wheel_length}" radius="${wheel_diam/2.0}"/>
+            <xacro:wheel_inertia/>
         </inertial>
     </link>
     <joint name="right_wheel_joint" type="continuous">
         <axis xyz="0 1 0"/>
-        <parent link="base_link"/>
+        <parent link="chassis_link"/>
         <child link="right_wheel"/>
-        <origin rpy="0 0 0" xyz="0 -0.43751887 -0.61759696"/>
+        <origin rpy="0 0 0" xyz="0 ${right_wheel_y} ${wheel_z}"/>
     </joint>
     <xacro:Transmission joint="right_wheel_joint"/>
@@ -102,13 +118,13 @@
         </collision>
         <inertial>
-            <mass value="1.0"/>
-            <xacro:cylinder_inertia mass="1.0" length="1.0" radius="1.0"/>
+            <mass value="${caster_mass}"/>
+            <xacro:caster_inertia/>
         </inertial>
     </link>
     <joint name="front_caster_joint" type="continuous">
         <axis xyz="0 0 1"/>
-        <parent link="base_link"/>
+        <parent link="chassis_link"/>
         <child link="front_caster"/>
-        <origin rpy="0 0 0" xyz="0.55951056 0 -0.619167561"/>
+        <origin rpy="0 0 0" xyz="${front_caster_x} 0 ${caster_z}"/>
     </joint>
     <link name="front_caster_wheel">
@@ -126,6 +142,6 @@
         </collision>
         <inertial>
-            <mass value="1.0"/>
-            <xacro:cylinder_inertia mass="1.0" length="1.0" radius="1.0"/>
+            <mass value="${caster_wheel_mass}"/>
+            <xacro:caster_wheel_inertia/>
         </inertial>
     </link>
@@ -134,5 +150,5 @@
         <parent link="front_caster"/>
         <child link="front_caster_wheel"/>
-        <origin rpy="0 0 0" xyz="0.03621719 0 -0.04361749"/>
+        <origin rpy="0 0 0" xyz="${front_caster_wheel_x} 0 ${caster_wheel_z}"/>
     </joint>
     <!-- Back caster wheel support -->
@@ -151,13 +167,13 @@
         </collision>
         <inertial>
-            <mass value="1.0"/>
-            <xacro:cylinder_inertia mass="1.0" length="1.0" radius="1.0"/>
+            <mass value="${caster_mass}"/>
+            <xacro:caster_inertia/>
         </inertial>
     </link>
     <joint name="back_caster_joint" type="continuous">
         <axis xyz="0 0 1"/>
-        <parent link="base_link"/>
+        <parent link="chassis_link"/>
         <child link="back_caster"/>
-        <origin rpy="0 0 0" xyz="-0.55951056 0 -0.619167561"/>
+        <origin rpy="0 0 0" xyz="${back_caster_x} 0 ${caster_z}"/>
     </joint>
     <link name="back_caster_wheel">
@@ -175,6 +191,6 @@
         </collision>
         <inertial>
-            <mass value="1.0"/>
-            <xacro:cylinder_inertia mass="1.0" length="1.0" radius="1.0"/>
+            <mass value="${caster_wheel_mass}"/>
+            <xacro:caster_wheel_inertia/>
         </inertial>
     </link>
@@ -183,5 +199,132 @@
         <parent link="back_caster"/>
         <child link="back_caster_wheel"/>
-        <origin rpy="0 0 0" xyz="-0.03621719 0 -0.04361749"/>
-    </joint>
+        <origin rpy="0 0 0" xyz="${back_caster_wheel_x} 0 ${caster_wheel_z}"/>
+    </joint>
+    <!-- Base laser / LIDAR -->
+    <link name="base_laser">
+        <visual>
+            <origin rpy="0 0 0" xyz="0 0 0"/>
+            <geometry>
+                <mesh filename="package://caffeine/urdf/meshes/hokuyo.dae"/>
+            </geometry>
+        </visual>
+        <collision>
+            <origin rpy="0 0 0" xyz="0 0 0"/>
+            <geometry>
+                <mesh filename="package://caffeine/urdf/meshes/hokuyo.dae"/>
+            </geometry>
+        </collision>
+        <inertial>
+            <mass value="${hokuyo_mass}"/>
+            <xacro:box_inertia mass="${hokuyo_mass}" length="${hokuyo_length}" width="${hokuyo_width}" height="${hokuyo_height}"/>
+        </inertial>
+    </link>
+    <joint name="base_laser_joint" type="fixed">
+        <parent link="base_link"/>
+        <child link="base_laser"/>
+        <origin xyz="${hokuyo_x} 0 0" rpy="0 0 0"/>
+    </joint>
+    <!-- ZED Camera -->
+    <link name="zed_camera_link">
+        <visual>
+            <origin xyz="0 0 0" rpy="0 0 0"/>
+            <!-- TODO: should be using the mesh but couldn't get it to work -->
+            <geometry>
+                <box size="${ZED_camera_width} ${ZED_camera_length} ${ZED_camera_height}"/>
+            </geometry>
+        </visual>
+        <collision>
+            <origin xyz="0 0 0" rpy="0 0 0"/>
+            <geometry>
+                <box size="${ZED_camera_width} ${ZED_camera_length} ${ZED_camera_height}"/>
+            </geometry>
+        </collision>
+        <inertial>
+            <mass value="${ZED_camera_mass}"/>
+            <xacro:box_inertia mass="${ZED_camera_mass}" length="${ZED_camera_length}" width="${ZED_camera_width}" height="${ZED_camera_height}"/>
+        </inertial>
+    </link>
+    <joint name="zed_camera_joint" type="fixed">
+        <parent link="stand_link"/>
+        <child link="zed_camera_link"/>
+        <origin xyz="${ZED_camera_x} 0 0" rpy="0 ${pi/4} 0"/>
+    </joint>
+   <!-- ZED camera lenses -->
+   <!-- NOTE: I'm only defining one and not visually showing any-->
+   <!-- I only need one for purposes of using the plugin -->
+   <!-- TODO: check if it's fine to call the left lense camera_link (rtabmap doesn't specify whether it wants the lense frame or the camera frame itself) -->
+   <link name="camera_link">
+       <!-- Inertial tag here to ensure that link does not phase through robot-->
+       <inertial>
+            <mass value="0.0001"/>
+            <inertia ixx="0.0001" ixy="0" ixz="0" iyy="0.0001" iyz="0" izz="0.00001"/>
+       </inertial>
+   </link>
+   <joint name="camera_link_joint" type="fixed">
+       <origin xyz="${ZED_camera_length/2.0} 0 0" rpy="0 0 0"/>
+       <parent link="zed_camera_link"/>
+       <child link="camera_link"/>
+   </joint>
+   <link name="camera_view_link">
+       <!-- Inertial tag here to ensure that link does not phase through robot-->
+       <inertial>
+            <mass value="0.0001"/>
+            <inertia ixx="0.0001" ixy="0" ixz="0" iyy="0.0001" iyz="0" izz="0.00001"/>
+       </inertial>
+   </link>
+   <joint name="camera_view_link_joint" type="fixed">
+       <origin xyz="0 0 0" rpy="${-pi/2} 0 ${-pi/2}"/>
+       <parent link="camera_link"/>
+       <child link="camera_view_link"/>
+   </joint>
+   <!-- IMU -->
+   <link name="imu_link">
+      <inertial>
+         <mass value="${phidget_mass}"/>
+         <xacro:box_inertia mass="${phidget_mass}" length="${phidget_length}" width="${phidget_width}" height="${phidget_height}"/>
+      </inertial>
+      <visual>
+         <origin xyz="0 0 0" rpy="0 0 0"/>
+         <geometry>
+            <box size="${phidget_length} ${phidget_width} ${phidget_height}"/>
+         </geometry>
+      </visual>
+      <collision>
+         <origin xyz="0 0 0" rpy="0 0 0"/>
+         <geometry>
+            <box size="${phidget_length} ${phidget_width} ${phidget_height}"/>
+         </geometry>
+      </collision>
+   </link>
+   <!-- IMU: attach imu_link to base_link -->
+   <joint name="base_link_to_imu_link" type="fixed">
+      <parent link="stand_link"/>
+      <child link="imu_link"/>
+      <origin xyz="0 0 0" rpy="0 0 0"/>
+   </joint>
+  <!-- GPS -->
+  <link name="gps_link">
+      <inertial>
+          <mass value="${gps_mass}"/>
+          <xacro:cylinder_inertia mass="${gps_mass}" length="${gps_length}" radius="${gps_diam / 2.0}"/>
+      </inertial>
+      <visual>
+          <origin xyz="0 0 0" rpy="0 0 0"/>
+          <geometry>
+              <cylinder length="${gps_length}" radius="${gps_diam / 2.0}"/>
+          </geometry>
+      </visual>
+      <collision>
+          <origin xyz="0 0 0" rpy="0 0 0"/>
+          <geometry>
+              <cylinder length="${gps_length}" radius="${gps_diam / 2.0}"/>
+          </geometry>
+      </collision>
+  </link>
+  <!-- GPS: attach gps_link to base_link -->
+  <joint name="gps_joint" type="fixed">
+      <parent link="stand_link"/>
+      <child link="gps_link"/>
+      <origin xyz="${gps_x} 0 0" rpy="0 0 0"/>
+  </joint>
 </robot>

File: slam-ws/src/caffeine/urdf/constants.xacro (robot description, xacro)
@@ -1,26 +1,34 @@
 <?xml version="1.0"?>
 <robot name="constants" xmlns:xacro="http://ros.org/wiki/xacro">
-   <!-- Constants for drivebase -->
-   <xacro:property name="base_length" value="1.268"/>
-   <xacro:property name="base_width" value="0.764"/>
-   <xacro:property name="base_height" value="0.01"/>
-   <xacro:property name="base_mass" value="39.091"/>
-   <!-- Constants for caster wheels -->
-   <xacro:property name="caster_wheel_diam" value="0.15"/>
-   <xacro:property name="caster_wheel_length" value="0.045"/>
-   <xacro:property name="caster_wheel_mass" value="1.0"/>
-   <xacro:property name="pi" value="3.1415926"/>
-   <xacro:property name="caster_wheel_z" value="-0.141"/>
-   <!-- Constants for side wheels -->
-   <xacro:property name="wheel_diam" value="0.25"/>
-   <xacro:property name="wheel_length" value="0.09"/>
-   <xacro:property name="wheel_mass" value="1.0"/>
-   <!-- Constants for casters -->
-   <xacro:property name="caster_length" value="0.113"/>
-   <xacro:property name="caster_width" value="0.089"/>
-   <xacro:property name="caster_height" value="0.141"/>
-   <xacro:property name="caster_x" value="0.578"/>
-   <xacro:property name="caster_z" value="-0.005"/>
-   <xacro:property name="caster_mass" value="1.0"/>
+    <!-- NOTE: -->
+    <!-- ALL coordinates relative to chassis_link UNLESS specified otherwise -->
+    <!-- TODO: modify the inertia and mass values -->
+    <!-- TODO: verify the wheel separation & wheel diam from mech -->
+    <xacro:property name="pi" value="3.1415826"/>
+    <!-- Base link constants -->
+    <xacro:property name="base_link_z" value="0.501747"/>
+    <!-- Stand link constants -->
+    <xacro:property name="stand_link_z" value="0.713459"/>
+    <!-- Constants for chassis_link -->
+    <xacro:property name="chassis_link_mass" value="30.0"/>
+    <!-- Constants for side wheels -->
+    <xacro:property name="wheel_mass" value="1.0"/>
+    <xacro:property name="wheel_separation" value="0.764"/>
+    <xacro:property name="wheel_diam" value="0.25"/>
+    <xacro:property name="left_wheel_y" value="0.43751887"/>
+    <xacro:property name="right_wheel_y" value="-0.43651887"/>
+    <xacro:property name="wheel_z" value="-0.61759696"/>
+    <!-- Constants for caster supports -->
+    <xacro:property name="caster_mass" value="1.0"/>
+    <xacro:property name="front_caster_x" value="0.55951056"/>
+    <xacro:property name="back_caster_x" value="-0.55951056"/>
+    <xacro:property name="caster_z" value="-0.619167561"/>
+    <!-- Constants for caster wheels -->
+    <xacro:property name="caster_wheel_mass" value="1.0"/>
+    <!-- These coordinates are relative to the front_caster frame -->
+    <xacro:property name="front_caster_wheel_x" value="0.03621719"/>
+    <xacro:property name="back_caster_wheel_x" value="-0.03621719"/>
+    <xacro:property name="caster_wheel_z" value="-0.04361749"/>
+   <!-- ALL the coordinates are located in reference to the specified coordinate frame -->
    <!-- Constants for hokuyo sensor -->
    <xacro:property name="hokuyo_length" value="0.05"/>
@@ -28,4 +36,6 @@
    <xacro:property name="hokuyo_height" value="0.07"/>
    <xacro:property name="hokuyo_mass" value="0.16"/>
+   <!-- Relative to base_link -->
+   <xacro:property name="hokuyo_x" value="0.55"/>
    <!-- Constants for Phidget IMU -->
    <xacro:property name="phidget_length" value="0.04"/>
@@ -33,19 +43,4 @@
    <xacro:property name="phidget_height" value="0.01"/>
    <xacro:property name="phidget_mass" value="0.04"/>
-   <!-- Constants for the basement -->
-   <xacro:property name="basement_height" value="0.103"/>
-   <xacro:property name="basement_width" value="0.305"/>
-   <xacro:property name="basement_length" value="0.456"/>
-   <xacro:property name="basement_mass" value="1.0"/>
-   <!-- Constants for the motor gearbox housing -->
-   <xacro:property name="gearbox_height" value="0.102"/>
-   <xacro:property name="gearbox_width" value="0.191"/>
-   <xacro:property name="gearbox_length" value="0.101"/>
-   <xacro:property name="gearbox_mass" value="0.1"/>
-  <!-- Constants for the stands -->
-  <xacro:property name="stand_length" value="0.412"/>
-  <xacro:property name="stand_width" value="0.254"/>
-  <xacro:property name="stand_height" value="1.324"/>
-  <xacro:property name="stand_mass" value="1.0"/>
   <!-- Constants for ZED camera -->
   <!-- NOTE: approx as a rectangular prism -->
@@ -54,4 +49,6 @@
   <xacro:property name="ZED_camera_width" value="0.03"/>
   <xacro:property name="ZED_camera_height" value="0.033"/>
+  <!-- Relative to stand_link -->
+  <xacro:property name="ZED_camera_x" value="0.177655"/>
   <!-- Constants for Garmin GPS -->
   <!-- NOTE: approx as a cylinder; garmin itself is similar to a hockey puck -->
@@ -59,3 +56,5 @@
   <xacro:property name="gps_length" value="0.0195"/>
   <xacro:property name="gps_mass" value="0.165"/>
+  <!-- Relative to stand link -->
+  <xacro:property name="gps_x" value="-0.10"/>
 </robot>

File: slam-ws/src/caffeine/urdf/inertias.xacro (robot description, xacro)
@@ -21,3 +21,31 @@
         />
     </xacro:macro>
+    <!-- Chassis link inertia -->
+    <xacro:macro name="chassis_link_inertia">
+        <inertia
+            ixx="1.0" ixy="0.0" ixz="0.0"
+            iyy="1.0" iyz="0.0" izz="1.0"
+        />
+    </xacro:macro>
+    <!-- Side wheel inertia -->
+    <xacro:macro name="wheel_inertia">
+        <inertia
+            ixx="1.0" ixy="0.0" ixz="0.0"
+            iyy="1.0" iyz="0.0" izz="1.0"
+        />
+    </xacro:macro>
+    <!-- Caster support inertia -->
+    <xacro:macro name="caster_inertia">
+        <inertia
+            ixx="1.0" ixy="0.0" ixz="0.0"
+            iyy="1.0" iyz="0.0" izz="1.0"
+        />
+    </xacro:macro>
+    <!-- Caster wheel inertia -->
+    <xacro:macro name="caster_wheel_inertia">
+        <inertia
+            ixx="1.0" ixy="0.0" ixz="0.0"
+            iyy="1.0" iyz="0.0" izz="1.0"
+        />
+    </xacro:macro>
 </robot>

Commit message: Slam 55 - Emulate ZED stereo cam in Simualtion (#111)
* Added new optical frame (zed_camera_link_optical)

* Moving camera to stand instead of base_link

* Removed viso2 and used rtab map's provided stereo_odometry node

* Integrated visual odometry into robot_localization

Co-authored-by: Federico Pizarro Bejarano <federico.pizarrobejarano@mail.utoronto.ca>

File: slam-ws/src/caffeine/urdf/caffeine.gazebo.xacro (robot description, xacro)
@@ -128,5 +128,5 @@
             <depthImageInfoTopicName>depth/camera_info</depthImageInfoTopicName>
             <pointCloudTopicName>depth/points</pointCloudTopicName>
-            <frameName>camera_view_link</frameName>
+            <frameName>zed_camera_link_optical</frameName>
             <hackBaseline>${ZED_camera_length}</hackBaseline>
             <distortionK1>0.0</distortionK1>

File: slam-ws/src/caffeine/urdf/caffeine.urdf.xacro (robot description, xacro)
@@ -306,7 +306,7 @@
    </link>
    <joint name="zed_camera_joint" type="fixed">
-       <parent link="base_link"/>
+       <parent link="stand"/>
        <child link="zed_camera_link"/>
-       <origin xyz="${stand_length/2} 0 ${stand_height + ZED_camera_height + base_height/2}" rpy="0 ${pi/4} 0"/>
+       <origin xyz="${stand_length/2} 0 ${stand_height + ZED_camera_height}" rpy="0 0 0"/>
    </joint>
    <!-- ZED camera lenses -->
@@ -326,15 +326,12 @@
        <child link="camera_link"/>
    </joint>
-   <link name="camera_view_link">
-       <!-- Inertial tag here to ensure that link does not phase through robot-->
-       <inertial>
-            <mass value="0.0001"/>
-            <inertia ixx="0.0001" ixy="0" ixz="0" iyy="0.0001" iyz="0" izz="0.00001"/>
-       </inertial>
-   </link>
-   <joint name="camera_view_link_joint" type="fixed">
+   <!-- Generate an optical frame http://www.ros.org/reps/rep-0103.html#suffix-frames so that ros and opencv can operate on the camera frame correctly -->
+   <link name="zed_camera_link_optical">
+   </link>
+   <joint name="zed_camera_link_optical_joint" type="fixed">
+       <!-- Transform b/w standard and optical frame -->
        <origin xyz="0 0 0" rpy="${-pi/2} 0 ${-pi/2}"/>
-       <parent link="camera_link"/>
-       <child link="camera_view_link"/>
+       <parent link="zed_camera_link"/>
+       <child link="zed_camera_link_optical"/>
    </joint>
    <!-- IMU -->
