Commit message: added sugar gearbox

File: slam-ws/src/proton/urdf/sugar_cube.gazebo.xacro (robot description, xacro)
@@ -1,5 +1,53 @@
 <?xml version="1.0"?>
 <robot name="sugar_cube_sim" xmlns:xacro="http://ros.org/wiki/xacro">
-    <link name="sugar_cube">
+   <xacro:include filename="$(find caffeine)/urdf/inertias.xacro"/>
+   <!-- Constants for drivebase -->
+   <xacro:property name="base_length" value="1.268"/>
+   <xacro:property name="base_width" value="0.764"/>
+   <xacro:property name="base_height" value="0.01"/>
+   <xacro:property name="base_mass" value="39.091"/>
+   <!-- Constants for side wheels -->
+   <xacro:property name="wheel_diam" value="0.25"/>
+   <xacro:property name="wheel_length" value="0.09"/>
+   <xacro:property name="wheel_mass" value="1.0"/>
+   <!-- Constants for the motor gearbox housing -->
+   <xacro:property name="gearbox_height" value="0.102"/>
+   <xacro:property name="gearbox_width" value="0.191"/>
+   <xacro:property name="gearbox_length" value="0.101"/>
+   <xacro:property name="gearbox_mass" value="0.1"/>
+    <!-- xacro macro for side wheels -->
+   <xacro:macro name="wheel_link_description">
+      <visual>
+         <origin rpy="${pi/2} 0 0" xyz="0 0 0"/>
+         <geometry>
+            <cylinder length="${wheel_length}" radius="${wheel_diam/2.0}"/>
+         </geometry>
+      </visual>
+      <collision>
+         <origin rpy="${pi/2} 0 0" xyz="0 0 0"/>
+         <geometry>
+            <cylinder length="${wheel_length}" radius="${wheel_diam/2.0}"/>
+         </geometry>
+      </collision>
+      <inertial>
+        <mass value="${wheel_mass}"/>
+        <xacro:cylinder_inertia mass="${wheel_mass}" length="${wheel_length}" radius="${wheel_diam/2}"/>
+      </inertial>
+   </xacro:macro>
+   <!-- Wheel motor definitions -->
+   <xacro:macro name="Transmission" params="joint">
+      <transmission name="trans_${joint}">
+         <type>transmission_interface/SimpleTransmission</type>
+         <joint name="${joint}">
+            <hardwareInterface>hardware_interface/EffortJointInterface</hardwareInterface>
+            <mechanicalReduction>1</mechanicalReduction>
+         </joint>
+         <actuator name="${joint}_motor">
+            <hardwareInterface>hardware_interface/EffortJointInterface</hardwareInterface>
+         </actuator>
+      </transmission>
+   </xacro:macro>
+    <!-- Base Sugar Cube -->
+    <link name="sugar_cube_base">
     <inertial>
         <origin xyz="0 0 0.5" rpy="0 0 0"/>
@@ -23,3 +71,16 @@
     </collision>
     </link>
+    <!-- Right side motor housing -->
+   <link name="right_sugar_gearbox">
+      <visual>
+         <origin rpy="0 0 0" xyz="0 0 ${-gearbox_height/2.0}"/>
+         <geometry>
+            <box size="${gearbox_length} ${gearbox_width} ${gearbox_height}"/>
+         </geometry>
+      </visual>
+   </link>
+   <joint name="base_to_right_leg" type="fixed">
+      <parent link="sugar_cube_base"/>
+      <child link="right_sugar_gearbox"/>
+   </joint>
 </robot>
